File: ai-camera-rev3.2.kicad_sch (KiCad schematic)
At the start: 176 parts, among them J1 Conn-01x02_P2mm_NONAME_JST-PH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, J2 TYPE-C-31-M-12, J3 MAXLAB, J4 Conn-02x10_P2.54mm_B-2100S20P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, J5 Conn-01x02_P1.25mm_10114829-1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, J6 Conn_01x24_FFC_0.5mm_AFC01-S2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, Q1 2N7002, Q10 2N7002, Q2 2N7002, Q3 AO3401A, Q4 AO3401A, Q5 2N7002, Q6 AO3401A, Q7 2N7002, Q8 AO3401A, Q9 2N7002, SW1 SW_PB_90deg_K2-1102AQ-H4CW-01, SW2 SW_PB_TS-1187A-B-A-B, SW3 SW_PB_TS-1187A-B-A-B, SW4 SW_PB_90deg_K2-1102AQ-H4CW-01, U1 TP4057-42-SOT26-R, U10 ESP32-S3-WROOM-1-N16R8, U11 MT9284-28J, U12 LTR-303ALS-01, U2 XC6206-2.8V, U3 PCF85063AT, U4 TI_SN74LVC1G373DBVR, U5 SY8089AAAC, U6 PIR_AS312, U7 XC6206-2.8V, U8 RT9166-12GVL, U9 AP1511B, Y1 32.768kHz_Q13FC1350000400

Commit message: updated poe schematic
Parts:
- removed C1, C11, C12, C25: 100u_CASE-B-3528_TAJB107K006RNJ, 00-kiml-capacitor-tantalum:CP_EIA-3528-15_AVX-H, symbol 00-kiml-capacitors-smd:100u_CASE-B-3528_TAJB107K006RNJ
- removed C10, C13, C14, C15, C16, C18, C19, C20, C24, C28, C29, C3, C33, C34, C37, C4, C41, C43, C45, C49, C5, C50, C51, C52, C55, C6, C7, C8, C9: 10u_0402_CL05A105KA5NQNC, Capacitor_SMD:C_0402_1005Metric, symbol 00-kiml-capacitors-smd:1u_0402_CL05A105KA5NQNC
- removed C17: 22p_0402_0402CG220J500NT, Capacitor_SMD:C_0402_1005Metric, symbol 00-kiml-capacitors-smd:22p_0402_0402CG220J500NT
- removed D1: 0603_RED_KT-0603R, LED_SMD:LED_0603_1608Metric, symbol 00-kiml-led-smd:0603_RED_KT-0603R
- removed D10, D11, D12, D13, D14, D15, D16, D17, D18, D9: 0603_IR_850nm_E6C0603IRAC1UDA, LED_SMD:LED_0603_1608Metric, symbol 00-kiml-led-smd:0603_IR_850nm_E6C0603IRAC1UDA
- removed D2: 0603_GREEN_19-217/GHC-YR1S2/3T, LED_SMD:LED_0603_1608Metric, symbol 00-kiml-led-smd:0603_GREEN_19-217/GHC-YR1S2/3T
- removed D3, D4, D5: SOD-523_BSD5C051L, Diode_SMD:D_SOD-523, symbol 00-kiml-power-protection:SOD-523_BSD5C051L
- removed D6, D8: B5819W-SL_SOD-123, Diode_SMD:D_SOD-123, symbol 00-kiml-diode:B5819W-SL_SOD-123
- removed J1: Conn-01x02_P2mm_NONAME_JST-PH_C47647, 00-kiml-connector-jst:JST_PH_S2B-PH-SM4-TB_1x02-1MP_P2.00mm_Horizontal, symbol 00-kiml-connector-jst:Conn-01x02_P2.0mm_NONAME_JST-PH_C47647
- removed J2: TYPE-C-31-M-12, 00-kiml-connector-usb:USB_C_Receptacle_HRO_TYPE-C-31-M-12, symbol 00-kiml-connector-usb:USB_C_Receptacle_USB2.0_TYPE-C-31-M-12
- removed J3: MAXLAB, Connector:Tag-Connect_TC2050-IDC-FP_2x05_P1.27mm_Vertical, symbol Connector_Generic:Conn_01x10
- removed J4: Conn-02x10_P2.54mm_B-2100S20P-B110, Connector_PinHeader_2.54mm:PinHeader_2x10_P2.54mm_Vertical, symbol 00-kiml-connector:Conn-02x10_P2.54mm_B-2100S20P-B110
- removed J5: Conn-01x02_P1.25mm_10114829-10102LF, 00-kiml-connector-amphenol:10114829-10102LF, symbol 00-kiml-connector:Conn-01x02_P1.25mm_10114829-10102LF
- removed JP1: USB_PWR, Jumper:SolderJumper-2_P1.3mm_Bridged2Bar_Pad1.0x1.5mm, symbol Jumper:SolderJumper_2_Bridged
- removed JP2: PIR, Jumper:SolderJumper-2_P1.3mm_Bridged2Bar_Pad1.0x1.5mm, symbol Jumper:SolderJumper_2_Bridged
- removed L1, L2: FB_2A_0805_220R@100MHz_BLM21PG221SN1D, Inductor_SMD:L_0805_2012Metric_Pad1.15x1.40mm_HandSolder, symbol 00-kiml-inductors:FB_2A_0805_220R@100MHz_BLM21PG221SN1D
- removed L3, L5: 10u_1.5A_4x4mm_SWPA4030S100MT, 00-kiml-inductor-smd:L_Sunlord_SWPA40xxS, symbol 00-kiml-inductors:10u_1.5A_4x4mm_SWPA4030S100MT
- removed Q1, Q10, Q2, Q5, Q7, Q9: 2N7002, Package_TO_SOT_SMD:SOT-23, symbol 00-kiml-transistor-fet:2N7002
- removed Q3, Q4, Q6, Q8: AO3401A, Package_TO_SOT_SMD:SOT-23, symbol 00-kiml-transistor-fet:AO3401A
- removed R1, R2, R23: 976k_0402_0402WGD9763TCE, Resistor_SMD:R_0402_1005Metric, symbol 00-kiml-resistors-smd:976k_0402_0402WGD9763TCE
- removed R10, R11, R12, R14, R20, R6, R7: 10k_0402_0402WGF1002TCE, Resistor_SMD:R_0402_1005Metric, symbol 00-kiml-resistors-smd:10k_0402_0402WGF1002TCE
- removed R13, R15, R16, R17, R18, R19, R21, R22, R24, R25, R31, R32: 215k_0402_0402WGD2153TCE, Resistor_SMD:R_0402_1005Metric, symbol 00-kiml-resistors-smd:215k_0402_0402WGD2153TCE
- removed R33: 2.43R_0805_0805W8F243KT5E, Resistor_SMD:R_0805_2012Metric, symbol 00-kiml-resistors-smd:2.43R_0805_0805W8F243KT5E
- removed R4, R5: 1k_0402_0402WGF1001TCE, Resistor_SMD:R_0402_1005Metric, symbol 00-kiml-resistors-smd:1k_0402_0402WGF1001TCE
- removed R8, R9: 5.1k_0603_0603WAF5101T5E, Resistor_SMD:R_0603_1608Metric, symbol 00-kiml-resistors-smd:5.1k_0603_0603WAF5101T5E
- removed SW1: SW_PB_90deg_K2-1102AQ-H4CW-01, 00-kiml-switch-button-tht:SW_PB_90deg_K2-1102AQ-H4CW-01, symbol 00-kiml-switch-button-tht:SW_PB_90deg_K2-1102AQ-N4CW-01
- removed U1: TP4057-42-SOT26-R, Package_TO_SOT_SMD:SOT-23-6, symbol 00-kiml-battery-management:TP4057-42-SOT26-R
- removed U11: MT9284-28J, Package_TO_SOT_SMD:SOT-23-6, symbol 00-kiml-driver-led:MT9284-28J
- removed U12: LTR-303ALS-01, 00-kiml-optical:Lite-On_LTR-303ALS-01, symbol 00-kiml-optical:LTR-303ALS-01
- removed U2: XC6206-2.8V, Package_TO_SOT_SMD:SOT-23, symbol 00-kiml-regulator-linear:XC6206-2.8V
- removed U3: PCF85063AT, Package_SO:SO-8_3.9x4.9mm_P1.27mm, symbol 00-kiml-timer-rtc:PCF85063AT/AAZ
- removed U4: TI_SN74LVC1G373DBVR, Package_TO_SOT_SMD:SOT-23-6, symbol 00-kiml-74xGxx:TI_SN74LVC1G373DBVR
- removed U5: SY8089AAAC, Package_TO_SOT_SMD:SOT-23-5, symbol 00-kiml-regulator-switching:SY8089AAAC
- removed U6: PIR_AS312, 00-kiml-optical:AS312, symbol 00-kiml-optical:PIR_AS312
- removed U9: AP1511B, Package_TO_SOT_SMD:SOT-23-6, symbol 00-kiml-ircut-driver:AP1511B
- removed Y1: 32.768kHz_Q13FC1350000400, 00-kiml-crystal-smd:Crystal_SMD_3215-2Pin_3.2x1.5mm, symbol 00-kiml-crystal:32.768kHz_Q13FC1350000400
- added R82, R83: 10k_0402_0402WGF1002TCE, Resistor_SMD:R_0402_1005Metric, symbol 00-kiml-resistors-smd:10k_0402_0402WGF1002TCE
- renumbered C26 to C73, C27 to C74, C2 to C75, C30 to C76, C31 to C77, C35 to C78, C36 to C79, C48 to C80, C53 to C81, C54 to C82, C56 to C83, C57 to C84, C21 to C85, C22 to C86, C23 to C87, C32 to C88, C38 to C89, C39 to C90, C40 to C91, C42 to C92, C44 to C93, C46 to C94, C47 to C95, D7 to D11, L4 to L9, R3 to R81, R26 to R84, R27 to R85, R28 to R86, R29 to R87, R30 to R88, SW2 to SW1, SW3 to SW2, SW4 to SW3, TP1 to TP14, TP2 to TP15, TP3 to TP16, TP4 to TP17, TP5 to TP18, TP6 to TP19, TP7 to TP20, TP8 to TP21, TP9 to TP22, TP10 to TP23, TP11 to TP24, TP12 to TP25, TP13 to TP26, TP14 to TP27, TP15 to TP28, TP16 to TP29, TP17 to TP30, TP18 to TP31, TP19 to TP32, TP20 to TP33, TP21 to TP34, TP22 to TP35, TP23 to TP36, TP24 to TP37, U7 to U16, U8 to U17, U10 to U18
Connections:
- net +3V3: now also R82.1, R83.1
- net CAM.SCL: now also R82.2
- net CAM.SDA: now also R83.2
- no-connect marks 12 -> 6
Other:
- note removed: "5K PROG sets charging current to 200 mA"
- note removed: "BATT_DETECT connected straight to the MCU, despite during the power-down condition they might supply some phantom current The hope is that output divider impedance is high enough for the phantom current to be low enough to cause any issue"
- note removed: "But it is better not to go any higher than 1M in divider resistors, since the output impedance of a divider will be significant enough to interplay with input ADC impedance of the MCU"
- note removed: "Dedicated power supply to support the PIR wakeup when main DC-DC is turned off"
- note removed: "External MAXLAB ESP32 programmer can be used to flash and interact with the camera via the TagConnect cable"
- note removed: "Given OV2640 sensitivity, an optimal LED should be C396643 @ LCSC (I_{max} ~40ma for T <= 60C, f_{peak} = 850nm, MPN: E6C0603IRAC1UDA) Forward drop should be in a region of ~1.6V The driver is capable of driving 7 white LEDs. WLED forward drop should be in the vicinity of ~3V. Meaning, that, hypotetically, we can drive up to 14 IR LEDs on this unit Shutdown current for U12 is 1uA"
- note removed: "I_{led} = [ V_{fb} = 94mV <->114mV ] / [ ~2.4R ] ~= 40mA"
- note removed: "Layout: Put IRCUT driver away from sensitive digital or analog lines"
- note removed: "Note: 3v3 and 5v are used as an output here to power the external programmer UART buffers. Internal programmer LDO output must be disabled then"
- note removed: "PWR_ON button starts DC-DC. MCU is responsible then for taking over PWR_EN signal The NMOS here is merely to make sure a signal polarity matches logical states (ON is HIGH>0V, OFF is LOW=0V) added benefit is that we no longer need OD MCU output on PWR_EN"
- note removed: "Pulling both inputs to 0 latches the state of the D-latch"
- note removed: "To prevent USB from powering VBUS completely, just in case"
- moved on the sheet: C73, C74, C76, C77, C78, C79, C80, C81, C82, C83, C84, C85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
