File: ESP32-PoE2_Rev_B.kicad_sch (KiCad schematic)
At the start: 119 parts, among them Q1 BC817-40(SOT23), Q2 BC817-40(SOT23), T1 LMUN2211LT1G(SOT-23), U1 BL4054B-42TPRN(SOT23-5), U2 CH340X(MSOP-10), U3 LAN8710A-EZC(QFN32), U4 SN74LVC1G04DBVR(SOT23-5), U5 SY8089AAAC(SOT23-5), U6 TPS2378DDAR(HSOIC-8), U7 TX4138(ESOIC-8), U8 TX4138(ESOIC-8)

Commit message: updated poe schematic
Parts:
- removed 24V_EN1: H-WX-1x2-LF, OLIMEX_Jumpers-FP:HN1x2(SMD)_H-WX-1x2-LF, symbol OLIMEX_Jumpers:JP1E
- removed 24V_EN1(Opened)1: MJ6, OLIMEX_Dummies-FP:MJ6, symbol OLIMEX_Jumpers:MJ6
- removed ACT1, CHRG1: LED/YELLOW/0603, OLIMEX_LEDs-FP:LED_0603_KA, symbol OLIMEX_Diodes:LED
- removed BAT1: DW02S, OLIMEX_Connectors-FP:LIPO_BAT_VERTICAL_DW02S, symbol OLIMEX_Connectors:BAT_CON
- removed BAT_SENS_E1: Opened, OLIMEX_Jumpers-FP:SJ, symbol OLIMEX_Jumpers:SJ
- removed C10, C11, C15, C5, C7: 100nF/10V/20%/X5R/C0402, OLIMEX_RLC-FP:C_0402_5MIL_DWS, symbol OLIMEX_RCL:C
- removed C14, C2, C4, C6: 22uF/6.3V/20%/X5R/C0603, OLIMEX_RLC-FP:C_0603_5MIL_DWS, symbol OLIMEX_RCL:C
- removed C18: 47uF/6.3V/20%/X5R/C0805, OLIMEX_RLC-FP:C_0805_5MIL_DWS, symbol OLIMEX_RCL:C
- removed C3: 1nF/2000V/10%/X7R/C1206, OLIMEX_RLC-FP:C_1206_5MIL_DWS_ISO, symbol OLIMEX_RCL:C
- removed D1, D4: 1N5822/SS34/SMA, OLIMEX_Diodes-FP:SMA-KA, symbol OLIMEX_Diodes:D_Schottky
- removed D2, D3, D5: 1N5819S4/SOD123, OLIMEX_Diodes-FP:SOD-123_1C-2A_KA, symbol OLIMEX_Diodes:D_Schottky
- removed D6: BAT54C(SOT23-3), OLIMEX_Diodes-FP:SOT23-3, symbol OLIMEX_Diodes:BAT54C(SOT23-3)
- removed FET1, FET2, FET3: WPM2015-3/TR, OLIMEX_Transistors-FP:SOT23, symbol OLIMEX_Transistors:P-MOS+DIOD
- removed L1: FB0805/600R/2A, OLIMEX_RLC-FP:L_0805_5MIL_DWS, symbol OLIMEX_RCL:L
- removed LAN_CON1: RJP-003TC1(LPJ4112CNL), OLIMEX_Connectors-FP:RJP-003TC1(LPJ4112CNL), symbol OLIMEX_Connectors:RJP-003TC1(LPJ4112CNL)
- removed LNK1: LED/GREEN/0603, OLIMEX_LEDs-FP:LED_0603_KA, symbol OLIMEX_Diodes:LED
- removed PWR1: LED/RED/0603, OLIMEX_LEDs-FP:LED_0603_KA, symbol OLIMEX_Diodes:LED
- removed Q1, Q2: BC817-40(SOT23), OLIMEX_Transistors-FP:SOT23, symbol OLIMEX_Transistors:Q_NPN_BEC
- removed R11, R12: 2.2k/R0402, OLIMEX_RLC-FP:R_0402_5MIL_DWS, symbol OLIMEX_RCL:R
- removed R22: 470k/R0402, OLIMEX_RLC-FP:R_0402_5MIL_DWS, symbol OLIMEX_RCL:R
- removed R23: 220R/R0402, OLIMEX_RLC-FP:R_0402_5MIL_DWS, symbol OLIMEX_RCL:R
- removed R24: 10k/R0402, OLIMEX_RLC-FP:R_0402_5MIL_DWS, symbol OLIMEX_RCL:R
- removed R25: 12k/1%/R0402, OLIMEX_RLC-FP:R_0402_5MIL_DWS, symbol OLIMEX_RCL:R
- removed R26: NA(2.2k/R0402), OLIMEX_RLC-FP:R_0402_5MIL_DWS, symbol OLIMEX_RCL:R
- removed R27: 220k/R0402, OLIMEX_RLC-FP:R_0402_5MIL_DWS, symbol OLIMEX_RCL:R
- removed R28: 49.9k/1%/R0402, OLIMEX_RLC-FP:R_0402_5MIL_DWS, symbol OLIMEX_RCL:R
- removed R29: 47k/R0402, OLIMEX_RLC-FP:R_0402_5MIL_DWS, symbol OLIMEX_RCL:R
- removed R30: 100k/R0402, OLIMEX_RLC-FP:R_0402_5MIL_DWS, symbol OLIMEX_RCL:R
- removed R4: 5.1k/1%/R0402, OLIMEX_RLC-FP:R_0402_5MIL_DWS, symbol OLIMEX_RCL:R
- removed RM1, RM2: RA1206_(4X0603)_4B8_2.2k, OLIMEX_RLC-FP:R_MATRIX_4, symbol OLIMEX_RCL:RA1206_(4x0603)_4B8_Smashed
- removed T1: LMUN2211LT1G(SOT-23), OLIMEX_Transistors-FP:SOT23, symbol OLIMEX_Transistors:LMUN2211LT1G(SOT-23)
- removed TVS1: ESDS314DBVR(SOT-23-5), OLIMEX_Diodes-FP:SOT-23-5, symbol OLIMEX_Diodes:ESDS314DBVR(SOT-23-5)
- removed TVS2, TVS3: NA(GG0402052R542P), OLIMEX_Diodes-FP:D_0402_5MIL_DWS, symbol OLIMEX_Diodes:GG0402052R542P
- removed U1: BL4054B-42TPRN(SOT23-5), OLIMEX_IC-FP:SOT-23-5, symbol OLIMEX_IC:BL4054B-42TPRN(SOT23-5)
- removed U2: CH340X(MSOP-10), OLIMEX_IC-FP:MSOP-10_Pitch-0.5mm_3.00x3.00x1.00mm, symbol OLIMEX_IC:CH340E(MSOP-10)
- removed U3: LAN8710A-EZC(QFN32), OLIMEX_IC-FP:QFN32_EP(33)_5.00x5.00x0.90mm_Pitch_0.50mm, symbol OLIMEX_IC:LAN8710A-EZC(QFN32)
- removed U4: SN74LVC1G04DBVR(SOT23-5), OLIMEX_IC-FP:SOT-23-5, symbol OLIMEX_IC:SN74LVC1G04DBVR(SOT23-5)
- removed U5: SY8089AAAC(SOT23-5), OLIMEX_Regulators-FP:SOT-23-5, symbol OLIMEX_IC:SY8009AAAC(SOT23-5)
- removed USB-UART1: USB-C-16P-F(A40-00119-A52-12), OLIMEX_Connectors-FP:USB2.0_TYPE-C(A40-00119-A52-12)_Paste, symbol OLIMEX_Connectors:USB2.0_TYPE-C(A40-00119-A52-12)
- added C10, C11, C14, C15, C34, C37: 22uF, Capacitor_SMD:C_0805_2012Metric, symbol Device:C
- added C18: 220uF/35V/20%8x12MM/LOW ESR, OLIMEX_RLC-FP:CPOL-RM3.5mm_8.0x11.5mm_PTH, symbol OLIMEX_RCL:CP
- added C19: 470uF/16V/20%/LOW_ESR/RM3.5/8x12MM, OLIMEX_RLC-FP:CPOL-RM3.5mm_8.0x11.5mm_PTH, symbol OLIMEX_RCL:CP
- added C2, C25: 10uF, Capacitor_SMD:C_0805_2012Metric, symbol Device:C
- added C21, C22, C23: 18pF, symbol Device:C
- added C26, C40, C41, C42, C43, C45, C48: 0.1uF, symbol Device:C
- added C29, C31, C46: 10nF, symbol Device:C
- added C3: 0.22uF, Capacitor_SMD:C_0603_1608Metric, symbol Device:C
- added C30, C6: 0.1uF, Capacitor_SMD:C_0603_1608Metric, symbol Device:C
- added C4: 1uF, Capacitor_SMD:C_0603_1608Metric, symbol Device:C
- added C44, C47, C50, C51, C55, C56: 10u_0402_CL05A105KA5NQNC, Capacitor_SMD:C_0402_1005Metric, symbol 00-kiml-capacitors-smd:1u_0402_CL05A105KA5NQNC
- added C49: 10uF, symbol Device:C
- added C5: 100uF/63V/20%/Low_ESR/RM5/10x13MM, OLIMEX_RLC-FP:CPOL-RM5mm_10.0x16.0mm_PTH, symbol OLIMEX_RCL:CP
- added C52: 22nF, symbol Device:C
- added C53, C54: 6.9nF, symbol Device:C
- added C7: DNP, Capacitor_SMD:C_0603_1608Metric, symbol Device:C
- added CR1, CR3: SMBJ15A, SMBJ15A:DO-214AASMB_J-BEND_LTF, symbol SMBJ15A:SMBJ15A
- added CR2: 7M-25.000MAAJ-T, CRYSTAL_TXC_7M, symbol 7M_25_000MAAJ_T:7M-25.000MAAJ-T
- added Class4_EN1: Closed, OLIMEX_Jumpers-FP:SJ_Closed, symbol OLIMEX_Jumpers:SJ_Closed
- added D1: SMAJ58A/SMA, OLIMEX_Diodes-FP:SMA-KA, symbol OLIMEX_Diodes:SMBJ6.0A
- added D2, D3, D4: SS54, SS34:DIOM7959X265N, symbol SS34:SS34
- added D5, D6: SS510/100V/5A/0.85V/DO214AB(SMC), OLIMEX_Diodes-FP:DO214AB(SMC)_1(K)-2(A), symbol OLIMEX_Diodes:D_Schottky_Small
- added F1: 2920L400_15MR, 2920L07560MR, symbol 2920L400_15MR:2920L400_15MR
- added IC1, IC2: SI4435DYPBF, SOIC127P600X175-8N, symbol SI4435DYPBF:SI4435DYPBF
- added IC3: KTA1170GVAE-TB, SON65P400X400X80-9N, symbol KTA1170GVAE-TB:KTA1170GVAE-TB
- added J1: B3B-XH-A, B3B-XH-A:JST_B3B-XH-A, symbol B3B-XH-A:B3B-XH-A
- added J2: ARJM11D7-114-AB-EW2, CONN_ARJM11D7-114-AB-EW2_ABR, symbol ARJM11D7_114_AB_EW2:ARJM11D7-114-AB-EW2
- added L1: SRP7028A-150M, SRP7028A:IND_SRP7028A_BRN, symbol SRP7028A:SRP7028A-1R8M
- added L3: 33uH/5.5A/60mR/20%/YSRH129-330M, OLIMEX_RLC-FP:HSMRH129_12.0x12.5x9.5(max), symbol OLIMEX_RCL:L
- added L4: MH1608-121Y, IND_BOURNS_MH1608, symbol BOURNS_MH1608:MH1608-121Y
- added L5: NRS5024T2R2NMGJ-2.2hF, NRS5024T2R2NMGJ:IND_NRS5024_TAY, symbol NRS5024T2R2NMGJ:NRS5024T2R2NMGJ
- added L8: FB_2A_0805_220R@100MHz_BLM21PG221SN1D, Inductor_SMD:L_0805_2012Metric_Pad1.15x1.40mm_HandSolder, symbol 00-kiml-inductors:FB_2A_0805_220R@100MHz_BLM21PG221SN1D
- added R11, R4: 100k, Resistor_SMD:R_0603_1608Metric, symbol Device:R
- added R12: 24.9k, Resistor_SMD:R_0603_1608Metric, symbol Device:R
- added R25, R48, R49, R50, R51: 0, Resistor_SMD:R_0603_1608Metric, symbol Device:R
- added R26: 1M, Resistor_SMD:R_0603_1608Metric, symbol Device:R
- added R37, R41, R42: 10k, Resistor_SMD:R_0603_1608Metric, symbol Device:R
- added R43: 63k 1%, Resistor_SMD:R_0603_1608Metric, symbol Device:R
- added R44: 20k 1%, Resistor_SMD:R_0603_1608Metric, symbol Device:R
- added R47: 12.4k 1%, Resistor_SMD:R_0603_1608Metric, symbol Device:R
- added R52, R54: 49.9 1%, Resistor_SMD:R_0603_1608Metric, symbol Device:R
- added R53, R55: 82 1%, Resistor_SMD:R_0603_1608Metric, symbol Device:R
- added R56: 10 1%, Resistor_SMD:R_0603_1608Metric, symbol Device:R
- added R57, R58: 330, Resistor_SMD:R_0603_1608Metric, symbol Device:R
- added TP1: 12V, TestPoint:TestPoint_Pad_D2.0mm, symbol Connector:TestPoint
- added TP2: 5VIN, TestPoint:TestPoint_Pad_D2.0mm, symbol Connector:TestPoint
- added TP3: 3V3, TestPoint:TestPoint_Pad_D2.0mm, symbol Connector:TestPoint
- added U1: TPS2378DDAR(HSOIC-8), OLIMEX_Regulators-FP:ESOIC-8, symbol OLIMEX_IC:TPS2378DDAR(HSOIC-8)
- added U10: XC6206-2.8V, Package_TO_SOT_SMD:SOT-23, symbol 00-kiml-regulator-linear:XC6206-2.8V
- added U11: RT9166-12GVL, Package_TO_SOT_SMD:SOT-23, symbol 00-kiml-regulator-linear:RT9166-12GVL
- added U2: LMR33630ADDAR, LMR33630ADDAR:VREG_LM5017MR_NOPB, symbol LMR33630ADDAR:LMR33630ADDAR
- added U3, U4: TX4138(ESOIC-8), OLIMEX_Regulators-FP:ESOIC-8, symbol OLIMEX_Regulators:TX4138(ESOIC-8)
- added U6: AP62201Z6-7, AP62201Z6_7:SOT563-Z6_1_DIO, symbol AP62201Z6_7:AP62201Z6-7
- added U9: W5500, W5500:QFP50P900X900X160-48N, symbol W5500:W5500
- C1: value 22uF/6.3V/20%/X5R/C0603 -> 100nF/100V/10%/X7R/C0603
- C12: value 2.2uF/6.3V/20%/X5R/C0402 -> 100nF/100V/10%/X7R/C0603; footprint OLIMEX_RLC-FP:C_0402_5MIL_DWS -> OLIMEX_RLC-FP:C_0603_5MIL_DWS; Fieldname 1 Value 1 -> (none); Fieldname2 Value2 -> (none); Fieldname3 Value3 -> (none)
- C13: value 100nF/10V/20%/X5R/C0402 -> 100nF/100V/10%/X7R/C0603; footprint OLIMEX_RLC-FP:C_0402_5MIL_DWS -> OLIMEX_RLC-FP:C_0603_5MIL_DWS; Fieldname 1 Value 1 -> (none); Fieldname2 Value2 -> (none); Fieldname3 Value3 -> (none)
- C16: value 1nF/NP0/50VDC/5%/C0603 -> 12pF/50V/5%/C0G/C0402; footprint OLIMEX_RLC-FP:C_0603_5MIL_DWS -> OLIMEX_RLC-FP:C_0402_5MIL_DWS; Fieldname 1 Value 1 -> (none); Fieldname2 Value2 -> (none); Fieldname3 Value3 -> (none)
- C17: value 1nF/50V/10%/X7R/C0402 -> 12pF/50V/5%/C0G/C0402; Fieldname 1 Value 1 -> (none); Fieldname2 Value2 -> (none); Fieldname3 Value3 -> (none)
- C8: value 100nF/10V/20%/X5R/C0402 -> NA(220pF/100V/C0603); footprint OLIMEX_RLC-FP:C_0402_5MIL_DWS -> OLIMEX_RLC-FP:C_0603_5MIL_DWS; Fieldname 1 Value 1 -> (none); Fieldname2 Value2 -> (none); Fieldname3 Value3 -> (none)
- C9: value 22uF/6.3V/20%/X5R/C0603 -> NA(220pF/100V/C0603); Fieldname 1 Value 1 -> (none); Fieldname2 Value2 -> (none); Fieldname3 Value3 -> (none)
- L2: value 2.2uH/1.5A/DCR=72mR/20%/3.00x3.00x1.50mm/CD32(NR3015T2R2M) -> 33uH/5.5A/60mR/20%/YSRH129-330M; footprint OLIMEX_RLC-FP:CD32 -> OLIMEX_RLC-FP:HSMRH129_12.0x12.5x9.5(max)
- R1: value 10k/R0402 -> 24.9k/1%/R0402; Fieldname 1 Value 1 -> (none); Fieldname2 Value2 -> (none); Fieldname3 Value3 -> (none)
- R10, R7, R8, R9: value 49.9R/1%/R0402 -> 0.03R/1%/R1206; footprint OLIMEX_RLC-FP:R_0402_5MIL_DWS -> OLIMEX_RLC-FP:R_1206_5MIL_DWS; Fieldname 1 Value 1 -> (none); Fieldname2 Value2 -> (none); Fieldname3 Value3 -> (none)
- R13: value 2.2k/R0402 -> 4.7R/R0402; Fieldname 1 Value 1 -> (none); Fieldname2 Value2 -> (none); Fieldname3 Value3 -> (none)
- R14: value 10k/R0402 -> 4.7R/R0402; Fieldname 1 Value 1 -> (none); Fieldname2 Value2 -> (none); Fieldname3 Value3 -> (none)
- R15: value 2.2k/R0402 -> NA(22R/R0603); footprint OLIMEX_RLC-FP:R_0402_5MIL_DWS -> OLIMEX_RLC-FP:R_0603_5MIL_DWS; Fieldname 1 Value 1 -> (none); Fieldname2 Value2 -> (none); Fieldname3 Value3 -> (none)
- R16: value 10k/R0402 -> NA(22R/R0603); footprint OLIMEX_RLC-FP:R_0402_5MIL_DWS -> OLIMEX_RLC-FP:R_0603_5MIL_DWS; Fieldname 1 Value 1 -> (none); Fieldname2 Value2 -> (none); Fieldname3 Value3 -> (none)
- R17: value 4.7k/R0402 -> 2.05k/1%/R0402; Fieldname 1 Value 1 -> (none); Fieldname2 Value2 -> (none); Fieldname3 Value3 -> (none)
- R18: value 2.2k/R0402 -> 2.05k/1%/R0402; Fieldname 1 Value 1 -> (none); Fieldname2 Value2 -> (none); Fieldname3 Value3 -> (none)
- R19: value 2.2k/R0402 -> 5.23k/1%/R0402; Fieldname 1 Value 1 -> (none); Fieldname2 Value2 -> (none); Fieldname3 Value3 -> (none)
- R2: value 1k/R0402 -> 1.27k/1%/62.5mW/R0402; Fieldname 1 Value 1 -> (none); Fieldname2 Value2 -> (none); Fieldname3 Value3 -> (none)
- R20: value 10R/R0402 -> 30.1k/1%/R0402; Fieldname 1 Value 1 -> (none); Fieldname2 Value2 -> (none); Fieldname3 Value3 -> (none)
- R21: value 470k/R0402 -> 30.1k/1%/R0402; Fieldname 1 Value 1 -> (none); Fieldname2 Value2 -> (none); Fieldname3 Value3 -> (none)
- R3: value 5.1k/1%/R0402 -> 66.5R/1%/125mW/R0805; footprint OLIMEX_RLC-FP:R_0402_5MIL_DWS -> OLIMEX_RLC-FP:R_0805_5MIL_DWS
- R5: value 10k/R0402 -> 9.1k/1W/R2512; footprint OLIMEX_RLC-FP:R_0402_5MIL_DWS -> OLIMEX_RLC-FP:R_2512_MM_DWS
- R6: value 2.2k/R0402 -> 9.1k/1W/R2512; footprint OLIMEX_RLC-FP:R_0402_5MIL_DWS -> OLIMEX_RLC-FP:R_2512_MM_DWS
- renumbered C19 to C20, C20 to C24, C21 to C27, C22 to C28, C23 to C32, C24 to C33, C25 to C35, C26 to C36, C27 to C38, C28 to C39, Class4_EN1 to Class4_EN2, L3 to L6, L4 to L7, R31 to R22, R32 to R23, R33 to R24, R34 to R27, R35 to R28, R36 to R29, R37 to R30, R38 to R31, R39 to R32, R40 to R33, R41 to R34, R42 to R35, R43 to R36, R44 to R38, R45 to R39, R46 to R40, R47 to R45, R48 to R46, U6 to U5
Connections:
- net +3.3VLAN is gone; now on an unnamed net: C8.1
- net GPIO16\I2C-SCL is gone; now on an unnamed net: R20.2
- net GPIO3\U0RXD is gone; now on an unnamed net: R15.2
- net RD+ is gone; now on net POE+: R8.2
- net RD- is gone; now on net POE+: R7.2
- net TD+ is gone; now on net POE+: R10.2
- net TD- is gone; now on net POE+: R9.2
- net VBAT is gone; now on net +5VP: R21.1
- net +5V: now also C25.2, D4.C, IC2.1 (S_1), IC2.2 (S_2), IC2.3 (S_3), U6.1 (VIN); no longer R5.1
- net +5VP: now also C17.1, C19.1 (+), D4.A, IC2.4 (G), L3.2
- net GND: now also R17.2, R18.2, R19.2, C10.2, C11.2, C14.2, C15.2, C18.2 (-), C19.2 (-), C2.2, C21.2, C22.2, C23.2, C25.1, C26.2, C29.2, C3.2, C31.2, C34.1, C37.1, C4.2, C40.2, C41.2, C42.2, C43.2, C44.2, C45.2, C46.2, C47.2, C48.2, C49.2, C5.2 (-), C50.2, C51.2, C52.2, C55.2, C56.2, CR1.2, CR2.2, CR2.4, D5.2 (A), D6.2 (A), IC3.9 (EP), J1.2, J1.3, R12.1, R44.1, R47.2, U1.5 (RTN), U1.8 (APD), U10.1 (GND), U11.1 (GND), U2.1 (PGND), U2.9 (AGND), U3.4 (GND), U4.4 (GND), U6.3 (GND), U9.14 (AGND__2), U9.16 (AGND__3), U9.19 (AGND__4), U9.29 (GND), U9.3 (AGND), U9.48 (AGND__5), U9.9 (AGND__1); no longer C12.2, C13.2, C16.1, C17.2, R16.2, R3.1
- net at L2.1: now also C12.1, D5.1 (K), U3.1 (SW)
- net at R13.1: now also U3.8 (BS)
- net at R13.2: now also C12.2
- net POE+: now reaches R6.1
- net POE+: now also C1.1, R1.1, R5.1, C5.1 (+), CR3.1, D1.1 (K), IC3.2 (VCC_1), IC3.3 (VCC_2), U1.1 (VDD), U3.3 (Vin), U4.3 (Vin)
- net at C13.1: now also R16.2, D6.1 (K), L3.1, U4.1 (SW); no longer C12.1
- net at C16.2: now also R17.1, R18.1, U3.5 (FB)
- net POE-: now reaches R2.2
- net POE-: now also C1.2, R3.1, CR3.2, D1.2 (A), IC3.6 (GND_1), IC3.7 (GND_2), U1.4 (VSS), U1.9 (EPAD)
- net at R16.1: now also C9.1
- net at R21.2: now also C17.2, R19.1, U4.5 (FB); no longer C17.1
- net at C35.2, R38.1, R45.2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: now also R39.1
- net at R14.2: now also C13.2
- removed net +3.3V: C1.1, L2.2, R1.1
- net +5V_USB: no longer names the net of R14.1
- net +5V_USB: now also U4.8 (BS)
- net CC2: no longer names the net of R3.2
- net CC2: now also Class4_EN1.1
- net GPIO33 renamed +12VP
- net +12VP: now also C16.1, L2.2, C18.1 (+), D2.A, IC1.4 (G)
- net VPP renamed 12VPP
- new net: C47.1, C50.1, C51.1, L8.2, U10.3 (VI), U11.3 (VI)
- new net: J2.13 (ANODE), R58.2
- new net: R37.1, U9.43 (PMODE2)
- new net: F1.1, J1.1
- new net: C4.1, R4.2
- new net: C30.1, L5.1, U6.2 (SW)
- new net: C30.2, U6.4 (BST)
- new net: R1.2, U1.2 (DEN)
- new net: Class4_EN1.2, R2.1, U1.3 (CLS)
- new net: U1.6 (CDB), U3.6 (EN), U4.6 (EN)
- new net: IC3.5 (IN4), J2.1 (VC2-)
- new net: J2.11 (ANODE), R57.2
- new net: IC3.8 (IN2), J2.2 (VC1-)
- new net: C54.2, J2.3 (RD-)
- new net: C46.1, J2.4 (RCT), R53.1, R55.1
- new net: C53.2, J2.5 (RD+)
- new net: IC3.4 (IN3), J2.6 (VC2+)
- new net: IC3.1 (IN1), J2.7 (VC1+)
- new net: C52.1, J2.9 (TCT), R56.1
- new net: R43.1, R44.2, U6.6 (FB)
- new net: R7.1, R8.1, U3.2 (ILIM), U3.9 (ILIM)
- new net: D3.A, F1.2
- new net: R10.1, R9.1, U4.2 (ILIM), U4.9 (ILIM)
- new net: C6.1, L1.1, U2.8 (SW)
- new net: C6.2, U2.7 (BOOT)
- new net: C7.2, R11.1, R12.2, U2.5 (FB)
- new net: C22.1, CR2.1, R26.1, U9.30 (XI)
- new net: C21.1, CR2.3, R25.2
- new net: R25.1, R26.2, U9.31 (XO)
- new net: R42.2, U9.45 (PMODE0)
- new net: C54.1, R50.2, R55.2
- new net: R50.1, U9.5 (RXN)
- new net: R41.1, U9.44 (PMODE1)
- new net +12V: D2.C, IC1.1 (S_1), IC1.2 (S_2), IC1.3 (S_3)
- new net +12VDC: C2.1, C3.1, CR1.1, D3.C, IC1.5 (D_1), IC1.6 (D_2), IC1.7 (D_3), IC1.8 (D_4), TP1.1, U2.2 (VIN), U2.3 (EN)
- new net +1V2: C56.1, U11.2 (VO)
- new net +2V8: C55.1, U10.2 (VO)
- new net +3.3VA: C40.1, C41.1, C42.1, C43.1, C45.1, C48.1, C49.1, L4.1, R52.2, R54.2, R56.2, U9.11 (AVDD__2), U9.15 (AVDD__3), U9.17 (AVDD__4), U9.21 (AVDD__5), U9.4 (AVDD), U9.8 (AVDD__1)
- new net +3V3: C23.1, C26.1, C34.2, C37.2, C44.1, L4.2, L5.2, L8.1, R37.2, R41.2, R42.1, R43.2, R57.1, R58.1, TP3.1, U9.28 (VDD)
- new net +5VDC: C10.1, C11.1, C14.1, C15.1, C7.1, IC2.5 (D_1), IC2.6 (D_2), IC2.7 (D_3), IC2.8 (D_4), L1.2, R11.2, TP2.1
- new net 1V2: C29.1, U9.22 (1V2O)
- new net ACTLED: J2.14 (CATHODE), U9.27 (ACTLED)
- new net EXRES1: R47.1, U9.10 (EXRES1)
- new net LINKLED: J2.12 (CATHODE), U9.25 (LINKLED)
- new net MISO: U9.34 (MISO)
- new net MOSI: U9.35 (MOSI)
- new net PG: R4.1, U2.4 (PG)
- new net RXP: C53.1, R51.1, R51.2, R53.2, U9.6 (RXP)
- new net SCLK: U9.33 (SCLK)
- new net TOCAP: C31.1, U9.20 (TOCAP)
- new net TXN: J2.8 (TD-), R48.1, R48.2, R52.1, U9.1 (TXN)
- new net TXP: J2.10 (TD+), R49.1, R49.2, R54.1, U9.2 (TXP)
- new net ~{INTn}: U9.36 (~{INTN})
- new net ~{RSTn}: U9.37 (~{RSTN})
- new net ~{SCSn}: U9.32 (~{SCSN})
- no-connect marks 10 -> 17
Other:
- note added: "3.3V Peak: 800 mA"
- note added: "Layout: Put LDOs as close as possible to the camera connector Keep separate "island" for camera connector and LDOs there"
- note removed: "!!!WARNING!!! When the board is powered via PoE, don't include the USB cable for to programming it!!! In case this is required, USB-ISO must be used for to guarantee galvanic isolation! See: https://www.olimex.com/Products/USB-Modules/USB-ISO/"
- note removed: "0"
- note removed: "1"
- note removed: "1.8V"
- note removed: "3.3V"
- note removed: "Any GPIO"
- note removed: "Auto program"
- note removed: "Battery Measurement"
- note removed: "Booting Mode"
- note removed: "Bootstrapping Pins Settings"
- note removed: "CHARGING"
- note removed: "DTR RTS->EN IO0"
- note removed: "Debugging Log on U0TXD During Booting"
- note removed: "Default"
- note removed: "Don't-care"
- note removed: "Download Boot"
- note removed: "EMAC"
- note removed: "EMAC_COL_out"
- note removed: "EMAC_CRS_out"
- note removed: "EMAC_MDC_out"
- note removed: "EMAC_MDI_in"
- note removed: "EMAC_MDO_out"
- note removed: "Ethernet"
- note removed: "External Power Sense"
- note removed: "Falling-edge:Input"
- note removed: "Falling-edge:Output"
- note removed: "For more information refer to esp_wroom_32_datasheet_en.pdf."
- note removed: "GPIO0"
- note removed: "GPIO0:"
- note removed: "GPIO12/MTDI"
- note removed: "GPIO15/MTDO"
- note removed: "GPIO2"
- note removed: "GPIO2:"
- note removed: "GPIO4:"
- note removed: "GPIO5"
- note removed: "GPIO5:"
- note removed: "General Purpose SPI"
- note removed: "HSPICLK_in/_out"
- note removed: "HSPID_in/_out"
- note removed: "HSPIQ_in/_out"
- note removed: "HSPI_CS0_in/_out"
- note removed: "HSPI_CS1_out"
- note removed: "HSPI_CS2_out"
- note removed: "I2C"
- note removed: "I2CEXT0_SCL_in"
- note removed: "I2CEXT0_SCL_out"
- note removed: "I2CEXT0_SDA_in"
- note removed: "I2CEXT0_SDA_out"
- note removed: "I2CEXT1_SCL_in"
- note removed: "I2CEXT1_SCL_out"
- note removed: "I2CEXT1_SDA_in"
- note removed: "I2CEXT1_SDA_out"
- note removed: "IBAT = 1000/Rprog = 100mA"
- note removed: "In RMII Mode"
- note removed: "Interface"
- note removed: "Internal Bootstrapping Resistors"
- note removed: "LiPo Charger"
- note removed: "MTDI/GPIO12:"
- note removed: "MTDO/GPIO15:"
- note removed: "Notes:"
- note removed: "Pin"
- note removed: "Power Supply"
- note removed: "Pull-Down"
- note removed: "Pull-Up"
- note removed: "Rising-edge:Input"
- note removed: "Rising-edge:Output"
- note removed: "Rprog"
- note removed: "SPI Flash Boot"
- note removed: "Signal"
- note removed: "Software Selectable Pins"
- note removed: "The PHY is setted up as follows: MODE: All capable(10/100Base) -Auto-negotiation enabled -RMII Configuration -SMI address: 0x00"
- note removed: "Timing of SDIO Slave"
- note removed: "U0TXD Silent"
- note removed: "U0TXD Toggling"
- note removed: "U8, C28 and R45 have to be Populated -> when WROVER is used, U8, C28 and R45 have to be NA -> when WROOM is used."
- note removed: "USB to UART"
- note removed: "VSPICLK_in/_out"
- note removed: "VSPID_in/_out"
- note removed: "VSPIQ_in/_out"
- note removed: "VSPI_CS0_in/_out"
- note removed: "VSPI_CS1_out"
- note removed: "VSPI_CS2_out"
- note removed: "Voltage of Internal LDO(VDD_SDIO)"
- note removed: "Vout=0.6*(1+Ra/Rb)"
- moved on the sheet: C20, C24, C27, C28, C32, C33, C35, C36, C38, C39, Class4_EN2, D7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

Commit message: GPIOs shouldn't have any conflicts
Parts:
- removed C20, C32, C33: 100nF/100V/10%/X7R/C0603, OLIMEX_RLC-FP:C_0603_5MIL_DWS, symbol OLIMEX_RCL:C
- removed C24: 100uF/63V/20%/Low_ESR/RM5/10x13MM, OLIMEX_RLC-FP:CPOL-RM5mm_10.0x16.0mm_PTH, symbol OLIMEX_RCL:CP
- removed C27, C28: NA(220pF/100V/C0603), OLIMEX_RLC-FP:C_0603_5MIL_DWS, symbol OLIMEX_RCL:C
- removed C35, C36: 12pF/50V/5%/C0G/C0402, OLIMEX_RLC-FP:C_0402_5MIL_DWS, symbol OLIMEX_RCL:C
- removed C38: 220uF/35V/20%8x12MM/LOW ESR, OLIMEX_RLC-FP:CPOL-RM3.5mm_8.0x11.5mm_PTH, symbol OLIMEX_RCL:CP
- removed C39: 470uF/16V/20%/LOW_ESR/RM3.5/8x12MM, OLIMEX_RLC-FP:CPOL-RM3.5mm_8.0x11.5mm_PTH, symbol OLIMEX_RCL:CP
- removed Class4_EN2: Closed, OLIMEX_Jumpers-FP:SJ_Closed, symbol OLIMEX_Jumpers:SJ_Closed
- removed D7: SMAJ58A/SMA, OLIMEX_Diodes-FP:SMA-KA, symbol OLIMEX_Diodes:SMBJ6.0A
- removed D8, D9: SS510/100V/5A/0.85V/DO214AB(SMC), OLIMEX_Diodes-FP:DO214AB(SMC)_1(K)-2(A), symbol OLIMEX_Diodes:D_Schottky_Small
- removed L6, L7: 33uH/5.5A/60mR/20%/YSRH129-330M, OLIMEX_RLC-FP:HSMRH129_12.0x12.5x9.5(max), symbol OLIMEX_RCL:L
- removed R22: 24.9k/1%/R0402, OLIMEX_RLC-FP:R_0402_5MIL_DWS, symbol OLIMEX_RCL:R
- removed R23: 1.27k/1%/62.5mW/R0402, OLIMEX_RLC-FP:R_0402_5MIL_DWS, symbol OLIMEX_RCL:R
- removed R24: 66.5R/1%/125mW/R0805, OLIMEX_RLC-FP:R_0805_5MIL_DWS, symbol OLIMEX_RCL:R
- removed R27, R28: 9.1k/1W/R2512, OLIMEX_RLC-FP:R_2512_MM_DWS, symbol OLIMEX_RCL:R
- removed R29, R30, R31, R32: 0.03R/1%/R1206, OLIMEX_RLC-FP:R_1206_5MIL_DWS, symbol OLIMEX_RCL:R
- removed R33, R34: 4.7R/R0402, OLIMEX_RLC-FP:R_0402_5MIL_DWS, symbol OLIMEX_RCL:R
- removed R35, R36: NA(22R/R0603), OLIMEX_RLC-FP:R_0603_5MIL_DWS, symbol OLIMEX_RCL:R
- removed R38, R39: 2.05k/1%/R0402, OLIMEX_RLC-FP:R_0402_5MIL_DWS, symbol OLIMEX_RCL:R
- removed R40: 5.23k/1%/R0402, OLIMEX_RLC-FP:R_0402_5MIL_DWS, symbol OLIMEX_RCL:R
- removed R45, R46: 30.1k/1%/R0402, OLIMEX_RLC-FP:R_0402_5MIL_DWS, symbol OLIMEX_RCL:R
- removed U5: TPS2378DDAR(HSOIC-8), OLIMEX_Regulators-FP:ESOIC-8, symbol OLIMEX_IC:TPS2378DDAR(HSOIC-8)
- removed U7, U8: TX4138(ESOIC-8), OLIMEX_Regulators-FP:ESOIC-8, symbol OLIMEX_Regulators:TX4138(ESOIC-8)
- C1: footprint OLIMEX_RLC-FP:C_0603_5MIL_DWS -> Capacitor_SMD:C_0603_1608Metric
- C21, C22, C23, C26, C29, C31, C40, C41, C42, C43, C45, C46, C48, C49: footprint (none) -> Capacitor_SMD:C_0603_1608Metric
- C52, C53, C54: footprint (none) -> Capacitor_SMD:C_1206_3216Metric
- CR2: footprint CRYSTAL_TXC_7M -> 7M_25_000MAAJ_T:CRYSTAL_TXC_7M
- F1: footprint 2920L07560MR -> 2920L400_15MR:2920L07560MR
- IC1, IC2: footprint SOIC127P600X175-8N -> SI4435DYPBF:SOIC127P600X175-8N
- IC3: footprint SON65P400X400X80-9N -> KTA1170GVAE-TB:SON65P400X400X80-9N
- J2: footprint CONN_ARJM11D7-114-AB-EW2_ABR -> ARJM11D7_114_AB_EW2:CONN_ARJM11D7-114-AB-EW2_ABR
- L4: footprint IND_BOURNS_MH1608 -> BOURNS_MH1608:IND_BOURNS_MH1608
- R1: value 24.9k/1%/R0402 -> 24.9k 1%
- R13: value 4.7R/R0402 -> 4.7
- R17, R18: value 2.05k/1%/R0402 -> 2.05k 1%
- R2: value 1.27k/1%/62.5mW/R0402 -> 1.27k 1% 62.5mW
- R20: value 30.1k/1%/R0402 -> 30.1k 1%
- R3: value 66.5R/1%/125mW/R0805 -> 66.5R 1% 125mW 0805
Connections:
- net PG renamed PGOOD
- no-connect marks 17 -> 14
Other:
- note removed: "PoE Power Supply"

Commit message: put all the components on the pcb on traces
Parts:
- removed C44, C47, C50, C51, C55, C56: 10u_0402_CL05A105KA5NQNC, Capacitor_SMD:C_0402_1005Metric, symbol 00-kiml-capacitors-smd:1u_0402_CL05A105KA5NQNC
- removed Class4_EN1: Closed, OLIMEX_Jumpers-FP:SJ_Closed, symbol OLIMEX_Jumpers:SJ_Closed
- removed L8: FB_2A_0805_220R@100MHz_BLM21PG221SN1D, Inductor_SMD:L_0805_2012Metric_Pad1.15x1.40mm_HandSolder, symbol 00-kiml-inductors:FB_2A_0805_220R@100MHz_BLM21PG221SN1D
- removed U10: XC6206-2.8V, Package_TO_SOT_SMD:SOT-23, symbol 00-kiml-regulator-linear:XC6206-2.8V
- removed U11: RT9166-12GVL, Package_TO_SOT_SMD:SOT-23, symbol 00-kiml-regulator-linear:RT9166-12GVL
- added C33: 10uF, Capacitor_SMD:C_0805_2012Metric, symbol Device:C
- added C35: 0.1uF, Capacitor_SMD:C_0603_1608Metric, symbol Device:C
- added C36, C38: 22uF, Capacitor_SMD:C_0805_2012Metric, symbol Device:C
- added L6: NRS5024T2R2NMGJ-2.2hF, NRS5024T2R2NMGJ:IND_NRS5024_TAY, symbol NRS5024T2R2NMGJ:NRS5024T2R2NMGJ
- added R30: 78k 1%, Resistor_SMD:R_0603_1608Metric, symbol Device:R
- added R31: 20k 1%, Resistor_SMD:R_0603_1608Metric, symbol Device:R
- added TP14: 3V9, TestPoint:TestPoint_Pad_D2.0mm, symbol Connector:TestPoint
- added U11: AP62201Z6-7, AP62201Z6_7:SOT563-Z6_1_DIO, symbol AP62201Z6_7:AP62201Z6-7
Connections:
- net +5V: now also C33.2, U11.1 (VIN)
- net GND: now also C33.1, C36.1, C38.1, R31.1, U11.3 (GND)
- net at R2.1, U1.3 (CLS): now also R3.2
- new net: R30.1, R31.2, U11.6 (FB)
- new net: C35.1, L6.1, U11.2 (SW)
- new net: C35.2, U11.4 (BST)
- new net +3V9: C36.2, C38.2, L6.2, R30.2, TP14.1
- no-connect marks 14 -> 15
Other:
- note added: "3.9V Peak: 1 A"
- note removed: "Layout: Put LDOs as close as possible to the camera connector Keep separate "island" for camera connector and LDOs there"
- moved on the sheet: C25, C30, C34, C37, L5, R43, R44, TP3, U6

Commit message: wip - started traces for layout
Parts:
- removed CR3: SMBJ15A, SMBJ15A:DO-214AASMB_J-BEND_LTF, symbol SMBJ15A:SMBJ15A
- added TP1: TestPoint, TestPoint:TestPoint_Pad_D2.0mm, symbol Connector:TestPoint
- added TP4, TP5: 3V3, TestPoint:TestPoint_Pad_D2.0mm, symbol Connector:TestPoint
- renumbered C21 to C20, C22 to C21, C23 to C22, C26 to C23, C25 to C24, C33 to C25, C29 to C26, C31 to C27, C30 to C28, C35 to C29, C34 to C30, C36 to C31, C37 to C32, C38 to C33, C40 to C34, C41 to C35, C42 to C36, C43 to C37, C45 to C38, C46 to C39, C48 to C40, C49 to C41, C52 to C42, C53 to C43, C54 to C44, R25 to R22, R26 to R23, R37 to R24, R41 to R25, R42 to R26, R43 to R27, R44 to R28, R30 to R29, R31 to R30, R47 to R31, R48 to R32, R49 to R33, R50 to R34, R51 to R35, R52 to R36, R53 to R37, R54 to R38, R55 to R39, R56 to R40, R57 to R41, R58 to R42, TP1 to TP2, TP2 to TP3, TP14 to TP6, TP3 to TP7, U6 to U5, U11 to U6, U9 to U7
Connections:
- net RXP is gone; now on net RX_P: C43.1, R35.1, R35.2, R37.2, U7.6 (RXP)
- net +12VP: now also TP4.1
- net +5VP: now also TP5.1
- net at C4.1, R4.2: now also U2.6 (VCC)
- net RX_N: now reaches C44.2, J2.3 (RD-)
- net RX_N: now also C44.1, R34.1, R34.2, R39.2, U7.5 (RXN)
- net RX_P: now reaches C43.2, J2.5 (RD+)
- net MISO renamed ETH_MISO
- net MOSI renamed ETH_MOSI
- net PGOOD: no longer names the net of R4.1, U2.4 (PG)
- net PGOOD: now also TP1.1
- net SCLK renamed ETH_SCLK
- net TXN renamed TX_N
- net TXP renamed TX_P
- net ~{INTn} renamed ~{ETH_INT}
- net ~{RSTn} renamed ~{ETH_RST}
- net ~{SCSn} renamed ~{ETH_CS}
Other:
- note added: "12V 3A 36W DC Barrel Jack"
- note added: "12V IN TO 5V BUCK"
- moved on the sheet: CR1, R41, R42
