File: expander.kicad_sch (KiCad schematic)
At the start: 16 parts, among them J5 B2B-PH-K-S, Q2 BSS138, U13 TPL5010, U5 MCP23017_ML

Commit message: put all the components on the pcb on traces
Parts:
- removed C20, C24: 0.1uF, Capacitor_SMD:C_0603_1608Metric, symbol Device:C
- removed D10: SMF33A, Diode_SMD:D_SMF, symbol Diode:SMF33A
- removed J5: B2B-PH-K-S, B2B-PH-K-S:JST_B2B-PH-K-S, symbol B2B-PH-K-S:B2B-PH-K-S
- removed Q2: BSS138, Package_TO_SOT_SMD:SOT-23, symbol Transistor_FET:BSS138
- removed R22, R23, R27, R28: 10k, Resistor_SMD:R_0603_1608Metric, symbol Device:R
- removed R24: 42.9k, Resistor_SMD:R_0603_1608Metric, symbol Device:R
- removed R67: 100, Resistor_SMD:R_0603_1608Metric, symbol Device:R
- removed S1: TS02-66-55-BK-160-LCR-D, TS02-66-55-BK-160-LCR-D:SW_TS02-66-55-BK-160-LCR-D, symbol TS02-66-55-BK-160-LCR-D:TS02-66-55-BK-160-LCR-D
- removed TP7: TestPoint, TestPoint:TestPoint_Pad_D2.0mm, symbol Connector:TestPoint
- removed U13: TPL5010, Package_TO_SOT_SMD:SOT-23-6, symbol Timer:TPL5010
- added C28: 0.1uF, Capacitor_SMD:C_0603_1608Metric, symbol Device:C
- added C32: 10uF, Capacitor_SMD:C_0805_2012Metric, symbol Device:C
- added J4: 5033981892, 5033981892:CONN_503398-1892_MOL, symbol 5033981892:5033981892
- added R29, R61, R65, R66: 10k, Resistor_SMD:R_0603_1608Metric, symbol Device:R
- added TP4: TestPoint, TestPoint:TestPoint_Pad_D2.0mm, symbol Connector:TestPoint
- C27: footprint (none) -> Capacitor_SMD:C_0603_1608Metric
Connections:
- net CAM.PWDN is gone; now on net MM_SYNC: U5.28 (GPB3)
- net LED is gone; now on net ~{RSTn}: U5.26 (GPB1)
- net SETUP is gone; now on net MM_SOP: U5.27 (GPB2)
- net +3V3: now also C28.1, C32.1, J4.4 (VDD), R29.1, R61.1, R65.2, R66.1
- net GND: now also C28.2, C32.2, J4.6 (VSS)
- net MM_SOP: no longer U5.20 (GPA3)
- net MM_SYNC: no longer U5.21 (GPA4)
- net ~{MM_RST}: now also U5.1 (GPB4); no longer U5.22 (GPA5)
- net ~{RSTn}: no longer U5.1 (GPB4)
- net ~{IO_RST}: now reaches U5.14 (~{RESET})
- net CAM.RST: no longer names the net of U5.2 (GPB5)
- net CAM.SCL renamed SCL
- net CAM.SDA renamed SDA
- net MM_CTS: no longer names the net of U5.23 (GPA6)
- net MM_RTS: no longer names the net of U5.24 (GPA7)
- new net CAM_SD_MISO: J4.7 (DA0), R29.2
- new net CAM_SD_MOSI: J4.3 (CMD), R61.2
- new net CAM_SD_SCK: J4.5 (CLK)
- new net SD_DETECT: J4.10 (DETECT_SWITCH), R65.1, TP4.1
- new net ~{SD_CS}: J4.2 (CD/DAT3), R66.2
Other:
- note added: "3.3V Peak: 200 mA Typ: 100 mA"
- note removed: "5 minutes"
- note removed: "5V PANEL LED W SERIES RESISTOR"

Commit message: wip - started traces for layout
Parts:
- removed TP4: TestPoint, TestPoint:TestPoint_Pad_D2.0mm, symbol Connector:TestPoint
- renumbered C27 to C59, C28 to C60, C32 to C61, J4 to J5, R29 to R61, R61 to R62, R65 to R63, R66 to R64, U5 to U12
Connections:
- net DF_BUSY: now reaches U12.20 (GPA3)
- net SPARE1: now reaches U12.21 (GPA4)
- net SPARE2: now reaches U12.22 (GPA5)
- net CAM_SD_SCK renamed CAM_SD_SCLK
- net ~{RSTn} renamed ETH_RST
Changed lines of the file:
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@@
-	)
-	(junction
-		(at 226.06 99.06)
-		(diameter 0)
-		(color 0 0 0 0)
 	)
 	(junction
@@
 	(wire
 		(pts
-			(xy 226.06 99.06) (xy 223.52 99.06)
+			(xy 223.52 99.06) (xy 237.49 99.06)
 		)
 		(stroke
@@
 	(wire
 		(pts
-			(xy 237.49 99.06) (xy 226.06 99.06)
-		)
-		(stroke
-			(width 0)
-			(type default)
-		)
-	)
-	(wire
-		(pts
 			(xy 102.87 90.17) (xy 92.71 90.17)
 		)
@@
 			(width 0)
 			(type default)
-		)
-	)
-	(label "~{SD_CS}"
-		(at 232.41 90.17 0)
-		(effects
-			(font
-				(size 1.27 1.27)
-			)
-			(justify left bottom)
 		)
 	)
@@
 			)
 			(justify right bottom)
-		)
-	)
-	(hierarchical_label "~{RSTn}"
-		(shape output)
-		(at 102.87 67.31 0)
-		(effects
-			(font
-				(size 1.27 1.27)
-			)
-			(justify left)
 		)
 	)
@@
 		)
 	)
+	(hierarchical_label "DF_BUSY"
+		(shape input)
+		(at 102.87 95.25 0)
+		(effects
+			(font
+				(size 1.27 1.27)
+			)
+			(justify left)
+		)
+	)
 	(hierarchical_label "~{MM_RST}"
 		(shape input)
@@
 		)
 	)
+	(hierarchical_label "SPARE2"
+		(shape input)
+		(at 102.87 100.33 0)
+		(effects
+			(font
+				(size 1.27 1.27)
+			)
+			(justify left)
+		)
+	)
 	(hierarchical_label "CAM_SD_MOSI"
 		(shape input)
@@
 		)
 	)
+	(hierarchical_label "SPARE1"
+		(shape input)
+		(at 102.87 97.79 0)
+		(effects
+			(font
+				(size 1.27 1.27)
+			)
+			(justify left)
+		)
+	)
 	(hierarchical_label "CAM_SD_MISO"
 		(shape output)
@@
 		)
 	)
-	(hierarchical_label "CAM_SD_SCK"
+	(hierarchical_label "CAM_SD_SCLK"
 		(shape input)
 		(at 232.41 86.36 0)
@@
 		(shape input)
 		(at 102.87 72.39 0)
+		(effects
+			(font
+				(size 1.27 1.27)
+			)
+			(justify left)
+		)
+	)
+	(hierarchical_label "ETH_RST"
+		(shape input)
+		(at 102.87 67.31 0)
+		(effects
+			(font
+				(size 1.27 1.27)
+			)
+			(justify left)
+		)
+	)
+	(hierarchical_label "~{SD_CS}"
+		(shape input)
+		(at 232.41 90.17 0)
 		(effects
 			(font
@@
 		(dnp no)
 		(fields_autoplaced yes)
-		(property "Reference" "#PWR049"
+		(property "Reference" "#PWR0102"
 			(at 95.25 60.96 0)
 			(effects
@@
 			(project ""
 				(path "/e0fc1b62-e519-47f0-a0fc-4ac6dbab9b04/a14327da-148b-4200-a87d-3de130f2539d"
-					(reference "#PWR049")
+					(reference "#PWR0102")
 					(unit 1)
 				)
@@
 		(on_board yes)
 		(dnp no)
-		(property "Reference" "C27"
+		(property "Reference" "C59"
 			(at 85.344 46.736 90)
 			(effects
@@
 			(project ""
 				(path "/e0fc1b62-e519-47f0-a0fc-4ac6dbab9b04/a14327da-148b-4200-a87d-3de130f2539d"
-					(reference "C27")
+					(reference "C59")
 					(unit 1)
 				)
@@
 		(on_board yes)
 		(dnp no)
-		(property "Reference" "C32"
+		(property "Reference" "C61"
 			(at 181.61 77.47 0)
 			(effects
@@
 			(project "LoiterGuardPcb"
 				(path "/e0fc1b62-e519-47f0-a0fc-4ac6dbab9b04/a14327da-148b-4200-a87d-3de130f2539d"
-					(reference "C32")
+					(reference "C61")
 					(unit 1)
 				)
@@
 		(on_board yes)
 		(dnp no)
-		(property "Reference" "R65"
+		(property "Reference" "R63"
 			(at 220.218 98.044 0)
 			(effects
@@
 			(project "LoiterGuardPcb"
 				(path "/e0fc1b62-e519-47f0-a0fc-4ac6dbab9b04/a14327da-148b-4200-a87d-3de130f2539d"
-					(reference "R65")
+					(reference "R63")
 					(unit 1)
 				)
@@
 		(on_board yes)
 		(dnp no)
-		(property "Reference" "R29"
+		(property "Reference" "R61"
 			(at 209.804 68.834 0)
 			(effects
@@
 			(project "LoiterGuardPcb"
 				(path "/e0fc1b62-e519-47f0-a0fc-4ac6dbab9b04/a14327da-148b-4200-a87d-3de130f2539d"
-					(reference "R29")
+					(reference "R61")
 					(unit 1)
 				)
@@
 		(dnp no)
 		(fields_autoplaced yes)
-		(property "Reference" "U5"
+		(property "Reference" "U12"
 			(at 77.0733 57.15 0)
 			(effects
@@
 			(project "LoiterGuardPcb"
 				(path "/e0fc1b62-e519-47f0-a0fc-4ac6dbab9b04/a14327da-148b-4200-a87d-3de130f2539d"
-					(reference "U5")
+					(reference "U12")
 					(unit 1)
 				)
@@
 		(dnp no)
 		(fields_autoplaced yes)
-		(property "Reference" "#PWR046"
+		(property "Reference" "#PWR0101"
 			(at 74.93 52.07 0)
 			(effects
@@
 			(project ""
 				(path "/e0fc1b62-e519-47f0-a0fc-4ac6dbab9b04/a14327da-148b-4200-a87d-3de130f2539d"
-					(reference "#PWR046")
+					(reference "#PWR0101")
 					(unit 1)
 				)
@@
 		(on_board yes)
 		(dnp no)
-		(property "Reference" "C28"
+		(property "Reference" "C60"
 			(at 173.99 77.47 0)
 			(effects
@@
 			(project "LoiterGuardPcb"
 				(path "/e0fc1b62-e519-47f0-a0fc-4ac6dbab9b04/a14327da-148b-4200-a87d-3de130f2539d"
-					(reference "C28")
+					(reference "C60")
 					(unit 1)
 				)
@@
 		(on_board yes)
 		(dnp no)
-		(property "Reference" "#PWR063"
+		(property "Reference" "#PWR0104"
 			(at 177.8 90.17 0)
 			(effects
@@
 			(project "LoiterGuardPcb"
 				(path "/e0fc1b62-e519-47f0-a0fc-4ac6dbab9b04/a14327da-148b-4200-a87d-3de130f2539d"
-					(reference "#PWR063")
+					(reference "#PWR0104")
 					(unit 1)
 				)
@@
 		(on_board yes)
 		(dnp no)
-		(property "Reference" "R61"
+		(property "Reference" "R62"
 			(at 219.202 69.596 0)
 			(effects
@@
 			(project "LoiterGuardPcb"
 				(path "/e0fc1b62-e519-47f0-a0fc-4ac6dbab9b04/a14327da-148b-4200-a87d-3de130f2539d"
-					(reference "R61")
+					(reference "R62")
 					(unit 1)
 				)
@@
 		(on_board yes)
 		(dnp no)
-		(property "Reference" "J4"
+		(property "Reference" "J5"
 			(at 199.898 68.834 0)
 			(effects
@@
 			(project "LoiterGuardPcb"
 				(path "/e0fc1b62-e519-47f0-a0fc-4ac6dbab9b04/a14327da-148b-4200-a87d-3de130f2539d"
-					(reference "J4")
+					(reference "J5")
 					(unit 1)
 				)
@@
 		(on_board yes)
 		(dnp no)
-		(property "Reference" "R66"
+		(property "Reference" "R64"
 			(at 229.362 69.596 0)
 			(effects
@@
 			(project "LoiterGuardPcb"
 				(path "/e0fc1b62-e519-47f0-a0fc-4ac6dbab9b04/a14327da-148b-4200-a87d-3de130f2539d"
-					(reference "R66")
+					(reference "R64")
 					(unit 1)
 				)
@@
 		(dnp no)
 		(fields_autoplaced yes)
-		(property "Reference" "#PWR089"
+		(property "Reference" "#PWR0103"
 			(at 177.8 69.85 0)
 			(effects
@@
 			(project "LoiterGuardPcb"
 				(path "/e0fc1b62-e519-47f0-a0fc-4ac6dbab9b04/a14327da-148b-4200-a87d-3de130f2539d"
-					(reference "#PWR089")
+					(reference "#PWR0103")
 					(unit 1)
 				)
@@
 		(dnp no)
 		(fields_autoplaced yes)
-		(property "Reference" "#PWR050"
+		(property "Reference" "#PWR0100"
 			(at 50.8 127 0)
 			(effects
@@
 			(project "LoiterGuardPcb"
 				(path "/e0fc1b62-e519-47f0-a0fc-4ac6dbab9b04/a14327da-148b-4200-a87d-3de130f2539d"
-					(reference "#PWR050")
+					(reference "#PWR0100")
 					(unit 1)
 				)
-			)
-		)
-	)
-	(symbol
-		(lib_id "Connector:TestPoint")
-		(at 226.06 99.06 180)
-		(unit 1)
-		(exclude_from_sim no)
-		(in_bom yes)
-		(on_board yes)
-		(dnp no)
-		(property "Reference" "TP4"
-			(at 224.282 105.156 0)
-			(effects
-				(font
-					(size 1.27 1.27)
-				)
-				(justify right)
-			)
-		)
-		(property "Value" "TestPoint"
-			(at 228.6 103.6319 0)
-			(effects
-				(font
-					(size 1.27 1.27)
-				)
-				(justify right)
-				(hide yes)
-			)
-		)
-		(property "Footprint" "TestPoint:TestPoint_Pad_D2.0mm"
-			(at 220.98 99.06 0)
-			(effects
-				(font
-					(size 1.27 1.27)
-				)
-				(hide yes)
-			)
-		)
-		(property "Datasheet" "~"
-			(at 220.98 99.06 0)
-			(effects
-				(font
-					(size 1.27 1.27)
-				)
-				(hide yes)
-			)
-		)
-		(property "Description" "test point"
-			(at 226.06 99.06 0)
-			(effects
-				(font
-					(size 1.27 1.27)
-				)
-				(hide yes)
-			)
-		)
-		(pin "1"
-		)
-		(instances
-			(project "LoiterGuardPcb"
-				(path "/e0fc1b62-e519-47f0-a0fc-4ac6dbab9b04/a14327da-148b-4200-a87d-3de130f2539d"
-					(reference "TP4")
-					(unit 1)
-				)
