File: LoiterGuardPcb.kicad_pcb (KiCad board)
At the start: 2 copper layers, 90 x 80 mm, 134 parts, among them J1 B6B-PH-SM4-TB, J2 5033981892, J3 B2B-PH-K-S, Q3 MBT3904DW1, Q4 BSS138, Q5 PDTC114EU_115, Q6 PDTC114EU_115, Q7 PDTC114EU_115, U10 TPL5010, U11 NL-SW-LTE-TC4NAG-B, U12 74AHC1G08, U13 XC6206-2.8V, U14 RT9166-12GVL, U15 AP1511B, U16 MT9284-28J, U9 ESP32-S3-WROOM-1-N16R8

Commit message: GPIOs shouldn't have any conflicts
Parts:
- removed C45, C46, C48, C49, C52, C53, C54: 10u_0402_CL05A105KA5NQNC, Capacitor_SMD:C_0402_1005Metric
- removed the C57 at (320.8, 74.6)
- removed the C58 at (320.8, 76.6)
- removed the C59 at (323.7, 64.8)
- removed the C60 at (323.7, 66.7)
- removed the C61 at (323.7, 68.7)
- removed the C62 at (323.7, 70.7)
- removed the C63 at (323.7, 72.6)
- removed the C64 at (323.7, 74.6)
- removed the C65 at (323.7, 76.6)
- removed the C66 at (326.6, 64.8)
- removed the C67 at (326.6, 66.7)
- removed the C68 at (326.6, 68.7)
- removed the C69 at (326.6, 70.7)
- removed D11: B5819W-SL_SOD-123, Diode_SMD:D_SOD-123
- removed D12, D13, D14, D15, D16, D17, D18, D19, D20, D21: 0603_IR_850nm_E6C0603IRAC1UDA, LED_SMD:LED_0603_1608Metric
- removed H1, H2, H3, H4: MountingHole_Pad, MountingHole:MountingHole_3.2mm_M3_Pad_TopBottom
- removed the R71 at (329.5, 81.7)
- removed the R72 at (337.0, 62.3)
- removed the TP11 at (318.1, 53.1)
- removed the TP12 at (318.1, 56.1)
- removed the TP13 at (318.1, 59.2)
- removed TP14, TP15, TP16, TP17, TP18, TP19, TP20, TP21, TP22, TP23, TP24, TP25, TP26, TP27, TP28, TP29, TP30, TP31, TP32, TP33, TP34: TestPoint, TestPoint:TestPoint_Pad_D1.0mm
- removed the U13 at (338.6, 66.2)
- removed the U14 at (338.6, 70.8)
- removed the U15 at (337.4, 54.0)
- removed U16: MT9284-28J, Package_TO_SOT_SMD:SOT-23-6
- added C10: 22uF, Capacitor_SMD:C_0805_2012Metric, F.Cu at (184.5, -0.16)
- added C100: 10u_0402_CL05A105KA5NQNC, Capacitor_SMD:C_0402_1005Metric, F.Cu at (264.4, 14.8)
- added C101: 10u_0402_CL05A105KA5NQNC, Capacitor_SMD:C_0402_1005Metric, F.Cu at (307.1, 2.50)
- added C11: 22uF, Capacitor_SMD:C_0805_2012Metric, F.Cu at (184.5, 2.85)
- added C14: 22uF, Capacitor_SMD:C_0805_2012Metric, F.Cu at (184.5, 5.86)
- added C15: 22uF, Capacitor_SMD:C_0805_2012Metric, F.Cu at (184.5, 8.87)
- added C2: 10uF, Capacitor_SMD:C_0805_2012Metric, F.Cu at (184.5, -3.17)
- added C25: 10uF, Capacitor_SMD:C_0805_2012Metric, F.Cu at (184.5, 11.9)
- added C3: 0.22uF, Capacitor_SMD:C_0603_1608Metric, F.Cu at (188.7, 19.7)
- added C30: 0.1uF, Capacitor_SMD:C_0603_1608Metric, F.Cu at (188.7, 29.8)
- added C34: 22uF, Capacitor_SMD:C_0805_2012Metric, F.Cu at (184.5, 14.9)
- added C37: 22uF, Capacitor_SMD:C_0805_2012Metric, F.Cu at (184.5, 17.9)
- added C4: 1uF, Capacitor_SMD:C_0603_1608Metric, F.Cu at (188.7, 22.2)
- added C44: 10u_0402_CL05A105KA5NQNC, Capacitor_SMD:C_0402_1005Metric, F.Cu at (208.2, 32.5)
- added C6: 0.1uF, Capacitor_SMD:C_0603_1608Metric, F.Cu at (188.7, 24.7)
- added C7: DNP, Capacitor_SMD:C_0603_1608Metric, F.Cu at (188.7, 27.2)
- added C96: 22p_0402_0402CG220J500NT, Capacitor_SMD:C_0402_1005Metric, F.Cu at (264.4, 6.91)
- added C97: 10u_0402_CL05A105KA5NQNC, Capacitor_SMD:C_0402_1005Metric, F.Cu at (264.4, 8.88)
- added C98: 10u_0402_CL05A105KA5NQNC, Capacitor_SMD:C_0402_1005Metric, F.Cu at (264.4, 10.8)
- added C99: 10u_0402_CL05A105KA5NQNC, Capacitor_SMD:C_0402_1005Metric, F.Cu at (264.4, 12.8)
- added CR1: SMBJ15A, SMBJ15A:DO-214AASMB_J-BEND_LTF, F.Cu at (227.1, 21.3)
- added CR2: 7M-25.000MAAJ-T, 7M_25_000MAAJ_T:CRYSTAL_TXC_7M, F.Cu at (199.0, 38.9)
- added CR3: SMBJ15A, SMBJ15A:DO-214AASMB_J-BEND_LTF, F.Cu at (227.1, 26.9)
- added D2: SS54, SS34:DIOM7959X265N, F.Cu at (212.2, -0.95)
- added D3: SS54, SS34:DIOM7959X265N, F.Cu at (212.2, 6.50)
- added D4: SS54, SS34:DIOM7959X265N, F.Cu at (212.2, 13.9)
- added F1: 2920L400_15MR, 2920L400_15MR:2920L07560MR, F.Cu at (223.4, -0.47)
- added H5: MountingHole_Pad, MountingHole:MountingHole_3.2mm_M3_Pad_TopBottom, F.Cu at (301.7, 3.50)
- added H6: MountingHole_Pad, MountingHole:MountingHole_3.2mm_M3_Pad_TopBottom, F.Cu at (301.7, 11.4)
- added H7: MountingHole_Pad, MountingHole:MountingHole_3.2mm_M3_Pad_TopBottom, F.Cu at (301.7, 19.4)
- added H8: MountingHole_Pad, MountingHole:MountingHole_3.2mm_M3_Pad_TopBottom, F.Cu at (301.7, 27.4)
- added IC1: SI4435DYPBF, SI4435DYPBF:SOIC127P600X175-8N, F.Cu at (207.0, 21.7)
- added IC2: SI4435DYPBF, SI4435DYPBF:SOIC127P600X175-8N, F.Cu at (207.0, 28.3)
- added IC3: KTA1170GVAE-TB, KTA1170GVAE-TB:SON65P400X400X80-9N, F.Cu at (219.3, 41.3)
- added J1: B3B-XH-A, B3B-XH-A:JST_B3B-XH-A, F.Cu at (124.9, 56.6)
- added J10: B2B-PH-K-S, B2B-PH-K-S:JST_B2B-PH-K-S, F.Cu at (166.2, 74.5)
- added J11: B16B-PH-SM4-TB_LF__SN_, B16B-PH-SM4-TB_LF__SN_:B16BPHSM4TBLFSN, F.Cu at (177.3, 88.9)
- added J12: 532610971, 532610971:CONN_532610001-SD_09_MOL, F.Cu at (161.1, 61.1)
- added J2: ARJM11D7-114-AB-EW2, ARJM11D7_114_AB_EW2:CONN_ARJM11D7-114-AB-EW2_ABR, F.Cu at (160.4, 117.7)
- added J6: FFC2B35-24-G_REVA2, FFC2B35-24-G_REVA2:GCT_FFC2B35-24-G_REVA2, F.Cu at (143.6, 91.6)
- added J7: B2B-PH-K-S, B2B-PH-K-S:JST_B2B-PH-K-S, F.Cu at (165.4, 81.2)
- added J8: B2B-PH-K-S, B2B-PH-K-S:JST_B2B-PH-K-S, F.Cu at (166.1, 88.2)
- added L1: SRP7028A-150M, SRP7028A:IND_SRP7028A_BRN, F.Cu at (221.1, 34.2)
- added L4: MH1608-121Y, BOURNS_MH1608:IND_BOURNS_MH1608, F.Cu at (228.8, 39.8)
- added L8: FB_2A_0805_220R@100MHz_BLM21PG221SN1D, Inductor_SMD:L_0805_2012Metric_Pad1.15x1.40mm_HandSolder, F.Cu at (213.6, 40.7)
- added Q6: AO3400A, Package_TO_SOT_SMD:SOT-23, F.Cu at (268.3, 8.32)
- added Q7: AO3400A, Package_TO_SOT_SMD:SOT-23, F.Cu at (268.3, 12.9)
- added R11: 100k, Resistor_SMD:R_0603_1608Metric, F.Cu at (188.7, 34.8)
- added R12: 24.9k, Resistor_SMD:R_0603_1608Metric, F.Cu at (192.7, 19.7)
- added R25: 0, Resistor_SMD:R_0603_1608Metric, F.Cu at (192.7, 22.2)
- added R26: 1M, Resistor_SMD:R_0603_1608Metric, F.Cu at (192.7, 24.7)
- added R37: 10k, Resistor_SMD:R_0603_1608Metric, F.Cu at (192.7, 27.2)
- added R4: 100k, Resistor_SMD:R_0603_1608Metric, F.Cu at (188.7, 32.3)
- added R41: 10k, Resistor_SMD:R_0603_1608Metric, F.Cu at (192.7, 29.8)
- added R42: 10k, Resistor_SMD:R_0603_1608Metric, F.Cu at (192.7, 32.3)
- added R43: 63k 1%, Resistor_SMD:R_0603_1608Metric, F.Cu at (192.7, 34.8)
- added R44: 20k 1%, Resistor_SMD:R_0603_1608Metric, F.Cu at (196.7, 19.7)
- added R47: 12.4k 1%, Resistor_SMD:R_0603_1608Metric, F.Cu at (196.7, 22.2)
- added R48: 0, Resistor_SMD:R_0603_1608Metric, F.Cu at (196.7, 24.7)
- added R49: 0, Resistor_SMD:R_0603_1608Metric, F.Cu at (196.7, 27.2)
- added R50: 0, Resistor_SMD:R_0603_1608Metric, F.Cu at (196.7, 29.8)
- added R51: 0, Resistor_SMD:R_0603_1608Metric, F.Cu at (196.7, 32.3)
- added R52: 49.9 1%, Resistor_SMD:R_0603_1608Metric, F.Cu at (196.7, 34.8)
- added R53: 82 1%, Resistor_SMD:R_0603_1608Metric, F.Cu at (200.7, 19.7)
- added R54: 49.9 1%, Resistor_SMD:R_0603_1608Metric, F.Cu at (200.7, 22.2)
- added R55: 82 1%, Resistor_SMD:R_0603_1608Metric, F.Cu at (200.7, 24.7)
- added R56: 10 1%, Resistor_SMD:R_0603_1608Metric, F.Cu at (200.7, 27.2)
- added R57: 330, Resistor_SMD:R_0603_1608Metric, F.Cu at (200.7, 29.8)
- added R58: 330, Resistor_SMD:R_0603_1608Metric, F.Cu at (200.7, 32.3)
- added R89: 100k, Resistor_SMD:R_0603_1608Metric, F.Cu at (196.1, 76.9)
- added R90: 100, Resistor_SMD:R_0603_1608Metric, F.Cu at (196.1, 79.4)
- added R91: 100k, Resistor_SMD:R_0603_1608Metric, F.Cu at (196.1, 81.9)
- added R92: 100, Resistor_SMD:R_0603_1608Metric, F.Cu at (196.1, 84.4)
- added R93: 215k_0402_0402WGD2153TCE, Resistor_SMD:R_0402_1005Metric, F.Cu at (307.1, 0.52)
- added TP1: 12V, TestPoint:TestPoint_Pad_D2.0mm, F.Cu at (204.8, 33.6)
- added TP2: 5VIN, TestPoint:TestPoint_Pad_D2.0mm, F.Cu at (204.8, 37.6)
- added TP3: 3V3, TestPoint:TestPoint_Pad_D2.0mm, F.Cu at (204.8, 41.7)
- added U10: XC6206-2.8V, Package_TO_SOT_SMD:SOT-23, F.Cu at (213.7, 32.3)
- added U11: RT9166-12GVL, Package_TO_SOT_SMD:SOT-23, F.Cu at (213.7, 37.0)
- added U19: DFR0299, DFR0299:MODULE_DFR0299, F.Cu at (112.6, 97.3)
- added U2: LMR33630ADDAR, LMR33630ADDAR:VREG_LM5017MR_NOPB, F.Cu at (191.5, 39.3)
- added U6: AP62201Z6-7, AP62201Z6_7:SOT563-Z6_1_DIO, F.Cu at (224.8, 40.2)
- added U9: W5500, W5500:QFP50P900X900X160-48N, F.Cu at (217.4, 24.2)
- L5: value FB_2A_0805_220R@100MHz_BLM21PG221SN1D -> NRS5024T2R2NMGJ-2.2hF; footprint Inductor_SMD:L_0805_2012Metric_Pad1.15x1.40mm_HandSolder -> NRS5024T2R2NMGJ:IND_NRS5024_TAY
- R69, R70: value 215k_0402_0402WGD2153TCE -> 10k_0402_0402WGF1002TCE
- U14: renamed from U11; moved to B.Cu
- moved L5 127.0 mm to (225.4, 14.4)
- moved C55 116.6 mm to (208.2, 40.4)
- moved C56 116.6 mm to (208.2, 42.4)
- moved C50 116.2 mm to (208.2, 36.5)
- moved C51 116.2 mm to (208.2, 38.5)
- moved C47 115.0 mm to (208.2, 34.5)
- moved J5 101.1 mm to (166.1, 94.2)
- moved R69 87.0 mm to (251.8, 38.4)
- moved R70 87.0 mm to (251.8, 40.4)
- moved J4 61.5 mm to (134.9, 120.6)
- moved U14 17.2 mm to (119.4, 95.6), turned to 180 degrees
- moved U12 12.7 mm to (142.9, 63.9)
- renumbered C29 to C57, C30 to C58, C31 to C59, C32 to C60, C33 to C61, C34 to C62, C35 to C63, C36 to C64, C37 to C65, C38 to C66, C39 to C67, C40 to C68, C41 to C69, C42 to C70, C43 to C71, C44 to C72, J1 to J3, J2 to J4, J3 to J5, Q3 to Q1, Q4 to Q2, Q5 to Q3, Q6 to Q4, Q7 to Q5, R49 to R59, R50 to R60, R51 to R61, R52 to R62, R53 to R63, R54 to R64, R55 to R65, R56 to R66, R57 to R67, R58 to R68, R59 to R71, R60 to R72, R61 to R73, R62 to R74, R63 to R75, R64 to R76, R65 to R77, R66 to R78, R67 to R79, R68 to R80, TP7 to TP10, TP8 to TP11, TP9 to TP12, TP10 to TP13, TP1 to TP4, TP2 to TP5, TP3 to TP6, TP4 to TP7, TP5 to TP8, TP6 to TP9, U9 to U12, U10 to U13, U12 to U15
Connections:
- C47 pad 1: +3.3VA -> Net-(U10-VI)
- C50 pad 1: +3.3VA -> Net-(U10-VI)
- C51 pad 1: +3.3VA -> Net-(U10-VI)
- C55 pad 1: +1V2 -> +2V8
- C56 pad 1: GND -> +1V2
- C56 pad 2: +3V3 -> GND
- L5 pad 1: +3V3 -> Net-(U6-SW)
- L5 pad 2: +3.3VA -> +3V3
- R69 pad 1: GNDPWR -> +3V3
- R69 pad 2: GND -> /MCU/CAM.SDA
- R70 pad 1: GND -> +3V3
- R70 pad 2: /CAM/IRCUT_CTRL -> /MCU/CAM.SCL

Commit message: put all the components on the pcb on traces
Parts:
- removed C100, C101, C47, C50, C51, C55, C56, C97, C98, C99: 10u_0402_CL05A105KA5NQNC, Capacitor_SMD:C_0402_1005Metric
- removed C58, C63, C69: 0.1uF, Capacitor_SMD:C_0603_1608Metric
- removed C59: 10uF, Capacitor_SMD:C_0805_2012Metric
- removed C96: 22p_0402_0402CG220J500NT, Capacitor_SMD:C_0402_1005Metric
- removed H5, H6, H7, H8: MountingHole_Pad, MountingHole:MountingHole_3.2mm_M3_Pad_TopBottom
- removed L8: FB_2A_0805_220R@100MHz_BLM21PG221SN1D, Inductor_SMD:L_0805_2012Metric_Pad1.15x1.40mm_HandSolder
- removed R60, R68, R71, R75, R76: 10k, Resistor_SMD:R_0603_1608Metric
- removed R73: 42.9k, Resistor_SMD:R_0603_1608Metric
- removed R93: 215k_0402_0402WGD2153TCE, Resistor_SMD:R_0402_1005Metric
- removed TP4, TP5, TP6: TestPoint, TestPoint:TestPoint_Pad_D2.0mm
- removed U10: XC6206-2.8V, Package_TO_SOT_SMD:SOT-23
- added C1: 100nF/100V/10%/X7R/C0603, Capacitor_SMD:C_0603_1608Metric, B.Cu at (130.3, 116.8)
- added C12: 100nF/100V/10%/X7R/C0603, OLIMEX_RLC-FP:C_0603_5MIL_DWS, B.Cu at (117.5, 108.5)
- added C13: 100nF/100V/10%/X7R/C0603, OLIMEX_RLC-FP:C_0603_5MIL_DWS, B.Cu at (126.7, 84.6)
- added C16: 12pF/50V/5%/C0G/C0402, OLIMEX_RLC-FP:C_0402_5MIL_DWS, B.Cu at (119.5, 121.6)
- added C17: 12pF/50V/5%/C0G/C0402, OLIMEX_RLC-FP:C_0402_5MIL_DWS, B.Cu at (116.5, 82.6)
- added C18: 220uF/35V/20%8x12MM/LOW ESR, OLIMEX_RLC-FP:CPOL-RM3.5mm_8.0x11.5mm_PTH, B.Cu at (120.2, 98.8)
- added C19: 470uF/16V/20%/LOW_ESR/RM3.5/8x12MM, OLIMEX_RLC-FP:CPOL-RM3.5mm_8.0x11.5mm_PTH, B.Cu at (139.4, 98.2)
- added C20: 0.1uF, Capacitor_SMD:C_0603_1608Metric, B.Cu at (142.1, 112.5)
- added C21: 18pF, Capacitor_SMD:C_0603_1608Metric, F.Cu at (151.0, 110.0)
- added C22: 18pF, Capacitor_SMD:C_0603_1608Metric, F.Cu at (157.2, 110.0)
- added C23: 18pF, Capacitor_SMD:C_0603_1608Metric, F.Cu at (147.7, 106.7)
- added C24: 0.1uF, Capacitor_SMD:C_0603_1608Metric, F.Cu at (158.6, 54.7)
- added C26: 0.1uF, Capacitor_SMD:C_0603_1608Metric, F.Cu at (149.3, 106.7)
- added C27: 0.1uF, Capacitor_SMD:C_0603_1608Metric, F.Cu at (134.0, 87.0)
- added C28: 0.1uF, Capacitor_SMD:C_0603_1608Metric, F.Cu at (132.6, 100.8)
- added C29: 10nF, Capacitor_SMD:C_0603_1608Metric, F.Cu at (145.3, 104.3)
- added C31: 10nF, Capacitor_SMD:C_0603_1608Metric, F.Cu at (145.2, 102.7)
- added C32: 10uF, Capacitor_SMD:C_0805_2012Metric, F.Cu at (130.8, 100.6)
- added C33: 10uF, Capacitor_SMD:C_0805_2012Metric, B.Cu at (175.8, 68.4)
- added C35: 0.1uF, Capacitor_SMD:C_0603_1608Metric, B.Cu at (169.2, 71.5)
- added C36: 22uF, Capacitor_SMD:C_0805_2012Metric, B.Cu at (179.3, 71.9)
- added C38: 22uF, Capacitor_SMD:C_0805_2012Metric, B.Cu at (177.3, 71.9)
- added C39: 470uF, Capacitor_THT:CP_Radial_D10.0mm_P5.00mm, F.Cu at (119.4, 67.2)
- added C40: 0.1uF, Capacitor_SMD:C_0603_1608Metric, F.Cu at (145.2, 99.4)
- added C41: 0.1uF, Capacitor_SMD:C_0603_1608Metric, F.Cu at (145.2, 97.9)
- added C42: 0.1uF, Capacitor_SMD:C_0603_1608Metric, F.Cu at (145.2, 96.4)
- added C43: 0.1uF, Capacitor_SMD:C_0603_1608Metric, F.Cu at (145.2, 94.9)
- added C45: 0.1uF, Capacitor_SMD:C_0603_1608Metric, F.Cu at (145.2, 93.4)
- added C46: 10nF, Capacitor_SMD:C_0603_1608Metric, F.Cu at (152.4, 81.1)
- added C48: 0.1uF, Capacitor_SMD:C_0603_1608Metric, F.Cu at (145.2, 91.9)
- added C49: 10uF, Capacitor_SMD:C_0603_1608Metric, F.Cu at (145.2, 90.4)
- added C5: 100uF/63V/20%/Low_ESR/RM5/10x13MM, OLIMEX_RLC-FP:CPOL-RM5mm_10.0x16.0mm_PTH, B.Cu at (129.9, 98.6)
- added C52: 22nF, Capacitor_SMD:C_1206_3216Metric, F.Cu at (161.2, 85.4)
- added C53: 6.9nF, Capacitor_SMD:C_1206_3216Metric, F.Cu at (150.9, 85.4)
- added C54: 6.9nF, Capacitor_SMD:C_1206_3216Metric, F.Cu at (154.4, 81.9)
- added C8: NA(220pF/100V/C0603), OLIMEX_RLC-FP:C_0603_5MIL_DWS, B.Cu at (105.0, 111.3)
- added C9: NA(220pF/100V/C0603), OLIMEX_RLC-FP:C_0603_5MIL_DWS, B.Cu at (136.2, 92.1)
- added D1: SMAJ58A/SMA, OLIMEX_Diodes-FP:SMA-KA, B.Cu at (130.3, 119.3)
- added D5: SS510/100V/5A/0.85V/DO214AB(SMC), OLIMEX_Diodes-FP:DO214AB(SMC)_1(K)-2(A), B.Cu at (113.2, 110.3)
- added D6: SS510/100V/5A/0.85V/DO214AB(SMC), OLIMEX_Diodes-FP:DO214AB(SMC)_1(K)-2(A), B.Cu at (131.5, 87.3)
- added J9: 878980204, 87898-0204:87898-0204_MOL, F.Cu at (123.3, 126.4)
- added L2: 33uH/5.5A/60mR/20%/YSRH129-330M, OLIMEX_RLC-FP:HSMRH129_12.0x12.5x9.5(max), B.Cu at (108.0, 99.1)
- added L3: 33uH/5.5A/60mR/20%/YSRH129-330M, OLIMEX_RLC-FP:HSMRH129_12.0x12.5x9.5(max), B.Cu at (144.2, 87.4)
- added L6: NRS5024T2R2NMGJ-2.2hF, NRS5024T2R2NMGJ:IND_NRS5024_TAY, B.Cu at (173.2, 73.9)
- added R1: 24.9k 1%, OLIMEX_RLC-FP:R_0402_5MIL_DWS, B.Cu at (131.0, 112.6)
- added R10: 0.03R/1%/R1206, OLIMEX_RLC-FP:R_1206_5MIL_DWS, B.Cu at (123.2, 93.1)
- added R13: 4.7, OLIMEX_RLC-FP:R_0402_5MIL_DWS, B.Cu at (117.5, 111.6)
- added R14: 4.7R/R0402, OLIMEX_RLC-FP:R_0402_5MIL_DWS, B.Cu at (126.7, 81.6)
- added R15: NA(22R/R0603), OLIMEX_RLC-FP:R_0603_5MIL_DWS, B.Cu at (108.0, 110.6)
- added R16: NA(22R/R0603), OLIMEX_RLC-FP:R_0603_5MIL_DWS, B.Cu at (136.2, 88.1)
- added R17: 2.05k 1%, OLIMEX_RLC-FP:R_0402_5MIL_DWS, B.Cu at (119.5, 119.1)
- added R18: 2.05k 1%, OLIMEX_RLC-FP:R_0402_5MIL_DWS, B.Cu at (119.5, 117.8)
- added R19: 5.23k/1%/R0402, OLIMEX_RLC-FP:R_0402_5MIL_DWS, B.Cu at (119.0, 82.6)
- added R2: 1.27k 1% 62.5mW, OLIMEX_RLC-FP:R_0402_5MIL_DWS, B.Cu at (128.7, 112.6)
- added R20: 30.1k 1%, OLIMEX_RLC-FP:R_0402_5MIL_DWS, B.Cu at (119.5, 120.3)
- added R21: 30.1k/1%/R0402, OLIMEX_RLC-FP:R_0402_5MIL_DWS, B.Cu at (117.7, 82.6)
- added R22: 10k, Resistor_SMD:R_0603_1608Metric, F.Cu at (167.4, 114.3)
- added R23: 10k, Resistor_SMD:R_0603_1608Metric, B.Cu at (142.1, 111.0)
- added R24: 42.9k, Resistor_SMD:R_0603_1608Metric, F.Cu at (158.1, 57.2)
- added R27: 10k, Resistor_SMD:R_0603_1608Metric, F.Cu at (161.9, 53.2)
- added R28: 10k, Resistor_SMD:R_0603_1608Metric, F.Cu at (165.0, 55.7)
- added R29: 10k, Resistor_SMD:R_0603_1608Metric, F.Cu at (134.2, 100.8)
- added R3: 66.5R 1% 125mW 0805, OLIMEX_RLC-FP:R_0805_5MIL_DWS, B.Cu at (128.8, 114.6)
- added R30: 78k 1%, Resistor_SMD:R_0603_1608Metric, B.Cu at (169.4, 69.0)
- added R31: 20k 1%, Resistor_SMD:R_0603_1608Metric, B.Cu at (172.7, 67.6)
- added R5: 9.1k/1W/R2512, OLIMEX_RLC-FP:R_2512_MM_DWS, B.Cu at (117.4, 87.7)
- added R6: 9.1k/1W/R2512, OLIMEX_RLC-FP:R_2512_MM_DWS, B.Cu at (113.0, 87.7)
- added R7: 0.03R/1%/R1206, OLIMEX_RLC-FP:R_1206_5MIL_DWS, B.Cu at (121.2, 107.8)
- added R8: 0.03R/1%/R1206, OLIMEX_RLC-FP:R_1206_5MIL_DWS, B.Cu at (121.2, 105.3)
- added R9: 0.03R/1%/R1206, OLIMEX_RLC-FP:R_1206_5MIL_DWS, B.Cu at (123.2, 90.4)
- added TP14: 3V9, TestPoint:TestPoint_Pad_D2.0mm, B.Cu at (178.0, 77.0)
- added U1: TPS2378DDAR(HSOIC-8), OLIMEX_Regulators-FP:ESOIC-8, B.Cu at (129.8, 107.9)
- added U3: TX4138(ESOIC-8), OLIMEX_Regulators-FP:ESOIC-8, B.Cu at (121.2, 113.3)
- added U4: TX4138(ESOIC-8), OLIMEX_Regulators-FP:ESOIC-8, B.Cu at (122.6, 85.3)
- added U5: MCP23017_ML, Package_DFN_QFN:QFN-28-1EP_6x6mm_P0.65mm_EP4.25x4.25mm, F.Cu at (138.5, 85.4)
- C10, C11, C14, C15, C2, C25, C3, C30, C34, C37, C4, C6, C62, C64, C65, C66, C67, C68, C7, C70, C72, CR1, D10, D2, D3, D4, F1, IC1, IC2, J1, J12, L1, L5, Q3, Q4, Q5, R11, R12, R4, R43, R44, R72, R74, R77, R79, S1, TP1, TP10, TP11, TP12, TP13, TP2, TP3, TP7, TP8, TP9, U2, U6: moved to B.Cu
- C44: value 10u_0402_CL05A105KA5NQNC -> 470uF; footprint Capacitor_SMD:C_0402_1005Metric -> Capacitor_THT:CP_Radial_D10.0mm_P5.00mm
- J6: value FFC2B35-24-G_REVA2 -> B6B-PH-SM4-TB; footprint FFC2B35-24-G_REVA2:GCT_FFC2B35-24-G_REVA2 -> B6B-PH-SM4-TB:JST_B6B-PH-SM4-TB
- U11: value RT9166-12GVL -> AP62201Z6-7; footprint Package_TO_SOT_SMD:SOT-23 -> AP62201Z6_7:SOT563-Z6_1_DIO; moved to B.Cu
- moved Q6 155.2 mm to (128.0, 74.9)
- moved Q7 150.0 mm to (123.8, 53.3), turned to 180 degrees
- moved Q5 143.9 mm to (124.8, 77.3), turned to 180 degrees
- moved Q4 143.7 mm to (124.9, 73.6), turned to 180 degrees
- moved Q3 143.7 mm to (125.0, 70.4), turned to 180 degrees
- moved TP8 143.3 mm to (127.3, 64.8), turned to 180 degrees
- moved TP13 143.1 mm to (128.9, 73.6), turned to 180 degrees
- moved R59 140.3 mm to (111.0, 93.2)
- moved R79 139.5 mm to (122.3, 78.6)
- moved C61 136.1 mm to (111.0, 94.7)
- moved C60 135.5 mm to (107.7, 94.5), turned to 180 degrees
- moved Q1 135.3 mm to (132.6, 79.9), turned to 90 degrees
- moved R72 134.1 mm to (127.2, 68.2)
- moved C57 133.8 mm to (113.3, 94.0), turned to 90 degrees
- moved TP11 133.4 mm to (140.4, 60.5), turned to 180 degrees
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Connections:
- net /MCU/RS485_RO renamed /MCU/CAM_SD_CLK
- net /MCU/VMON renamed /MCU/LED2
- net /MCU/WATER_PULSES renamed /MCU/~{INTn}
- net /MCU/~{ADC_CS} renamed /MCU/DF_RX
- net /MCU/~{DRDY_RTD_UP} renamed /MCU/DF_TX
- net /MCU/~{RTD_DN_CS} renamed /MCU/MM_CTS
- net /Outputs/CAM.D2 renamed /Outputs/~{CAM_CS}
- net /Outputs/CAM.D3 renamed /Outputs/CAM_SD_MISO
- net /Outputs/CAM.D4 renamed /Outputs/CAM_SD_SCLK
- net /Outputs/CAM.D5 renamed /Outputs/CAM_SD_MOSI
- net PG renamed /Poe/PGOOD
- C44 pad 1: +3V3 -> GND
- C44 pad 2: GND -> +12V
- J4 pad 10: /MCU/SD_DETECT -> /Expander/SD_DETECT
- J4 pad 2: /MCU/~{SD_CS} -> /Expander/~{SD_CS}
- J4 pad 3: /MCU/MOSI -> /Expander/CAM_SD_MOSI
- J4 pad 5: /MCU/SCK -> /Expander/CAM_SD_SCK
- J4 pad 7: /MCU/MISO -> /Expander/CAM_SD_MISO
- J6 pad 1: unconnected-(J6-Pad1) -> +3V3
- J6 pad 2: unconnected-(J6-Pad2) -> GND
- R61 pad 2: /MCU/MOSI -> /Expander/CAM_SD_MOSI
- R65 pad 1: /MCU/SD_DETECT -> /Expander/SD_DETECT
- R66 pad 2: /MCU/~{SD_CS} -> /Expander/~{SD_CS}
- R69 pad 2: /MCU/CAM.SDA -> /MCU/SDA
- R70 pad 2: /MCU/CAM.SCL -> /MCU/SCL
- U11 pad 1: GND -> +5V
- U11 pad 2: +1V2 -> Net-(U11-SW)
- U11 pad 3: Net-(U10-VI) -> GND
- U12 pad 10: /MCU/CELL_RX -> /MCU/CELL_TX
- U12 pad 11: /MCU/CELL_TX -> /MCU/CELL_RX
- U12 pad 13: /MCU/CELL_RST -> /MCU/USB-
- U12 pad 14: /MCU/CELL_CTS -> /MCU/USB+
- U12 pad 15: GND -> /MCU/LED1
- U12 pad 16: /MCU/~{DRDY_RTD_DN} -> /MCU/LED
- U12 pad 17: unconnected-(U12-IO9-Pad17) -> /MCU/MM_RTS
- U12 pad 18: unconnected-(U12-IO10-Pad18) -> /MCU/ETH_CS
- U12 pad 19: unconnected-(U12-IO11-Pad19) -> /MCU/ETH_MOSI
- U12 pad 20: unconnected-(U12-IO12-Pad20) -> /MCU/ETH_SCLK
- U12 pad 21: unconnected-(U12-IO13-Pad21) -> /MCU/ETH_MISO
- U12 pad 22: unconnected-(U12-IO14-Pad22) -> /MCU/CELL_RTS
- U12 pad 24: unconnected-(U12-IO47-Pad24) -> /MCU/SDA
- U12 pad 25: unconnected-(U12-IO48-Pad25) -> /MCU/SCL
- U12 pad 26: /MCU/CELL_RTS -> /MCU/~{IO_RST}
- U12 pad 28: /MCU/RS485_DI -> unconnected-(U12-IO35-Pad28)
- U12 pad 29: /MCU/~{SD_CS} -> unconnected-(U12-IO36-Pad29)
- U12 pad 30: /MCU/WD_DONE -> unconnected-(U12-IO37-Pad30)
- U12 pad 32: /MCU/SCK -> /MCU/CAM_SD_MOSI
- U12 pad 33: /MCU/MISO -> /MCU/CAM_SD_MISO
- U12 pad 34: unconnected-(U12-IO41-Pad34) -> /MCU/~{CAM_CS}
- U12 pad 35: /MCU/LED -> /MCU/~{SD_CS}
- U12 pad 38: /MCU/SETUP -> /MCU/MM_TX
- U12 pad 39: /MCU/MOSI -> /MCU/MM_RX
- U12 pad 4: unconnected-(U12-IO4-Pad4) -> /MCU/SETUP
- U12 pad 6: /MCU/SD_DETECT -> /MCU/LED3
- U12 pad 8: /MCU/~{RTD_UP_CS} -> /MCU/CELL_CTS
- U19 pad 1: +5V -> +3V3

Commit message: wip - started traces for layout
Parts:
- removed CR3: SMBJ15A, SMBJ15A:DO-214AASMB_J-BEND_LTF
- removed the J9 at (123.3, 126.4)
- added J10: 878980204, 87898-0204:87898-0204_MOL, F.Cu at (125.4, 102.9)
- added TP1: TestPoint, TestPoint:TestPoint_Pad_D2.0mm, B.Cu at (177.3, 97.5)
- added TP4: 3V3, TestPoint:TestPoint_Pad_D2.0mm, B.Cu at (116.4, 104.0)
- added TP5: 3V3, TestPoint:TestPoint_Pad_D2.0mm, B.Cu at (148.6, 95.9)
- IC3: moved to B.Cu
- moved R40 37.6 mm to (144.2, 120.7), turned to -90 degrees
- moved C42 35.7 mm to (144.2, 116.8)
- moved C39 32.1 mm to (161.1, 111.9), turned to 0 degrees
- moved IC3 26.7 mm to (139.5, 117.2), turned to 90 degrees
- moved C44 26.6 mm to (154.6, 108.4), turned to 0 degrees
- moved R37 25.7 mm to (158.8, 111.2), turned to 90 degrees
- moved C61 25.3 mm to (117.5, 122.1)
- moved R62 25.3 mm to (119.4, 125.4)
- moved R63 25.3 mm to (122.6, 122.4)
- moved C60 25.3 mm to (119.3, 122.4)
- moved R61 25.3 mm to (121.0, 122.3)
- moved R64 25.3 mm to (121.0, 125.4)
- moved R39 25.0 mm to (154.0, 111.2)
- moved R36 24.8 mm to (147.7, 109.1), turned to 180 degrees
- moved J6 24.5 mm to (182.5, 80.4)
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- renumbered C21 to C20, C22 to C21, C23 to C22, C26 to C23, C25 to C24, C33 to C25, C29 to C26, C31 to C27, C30 to C28, C35 to C29, C34 to C30, C36 to C31, C37 to C32, C38 to C33, C40 to C34, C41 to C35, C42 to C36, C43 to C37, C45 to C38, C46 to C39, C48 to C40, C49 to C41, C52 to C42, C53 to C43, C54 to C44, C57 to C45, C60 to C46, C61 to C47, C62 to C48, C20 to C49, C64 to C50, C65 to C51, C66 to C52, C67 to C53, C68 to C54, C24 to C55, C70 to C56, C71 to C57, C72 to C58, C27 to C59, C28 to C60, C32 to C61, C39 to C62, C44 to C63, D10 to D7, J5 to J4, J4 to J5, J7 to J6, J6 to J7, J10 to J9, R25 to R22, R26 to R23, R37 to R24, R41 to R25, R42 to R26, R43 to R27, R44 to R28, R30 to R29, R31 to R30, R47 to R31, R48 to R32, R49 to R33, R50 to R34, R51 to R35, R52 to R36, R53 to R37, R54 to R38, R55 to R39, R56 to R40, R57 to R41, R58 to R42, R59 to R43, R62 to R44, R63 to R45, R64 to R46, R67 to R47, R22 to R48, R69 to R49, R70 to R50, R23 to R51, R72 to R52, R24 to R53, R74 to R54, R27 to R55, R28 to R56, R77 to R57, R78 to R58, R79 to R59, R80 to R60, R29 to R61, R61 to R62, R65 to R63, R66 to R64, R89 to R65, R90 to R66, R91 to R67, R92 to R68, TP9 to TP10, TP10 to TP11, TP11 to TP12, TP12 to TP13, TP13 to TP14, TP1 to TP2, TP2 to TP3, TP14 to TP6, TP3 to TP7, TP7 to TP8, TP8 to TP9, U14 to U10, U15 to U11, U5 to U12, U19 to U13, U6 to U5, U11 to U6, U9 to U7, U12 to U8, U13 to U9
Connections:
- net /Poe/PGOOD renamed Net-(U2-PG)
- net /Poe/TXN renamed /Poe/TX_N
- net /Poe/TXP renamed /Poe/TX_P
- C4 pad 1: Net-(C4-Pad1) -> Net-(U2-VCC)
- C43 pad 1: /Poe/RXP -> /Poe/RX_P
- C43 pad 2: Net-(J2-RD+) -> /Poe/RX_P
- C44 pad 1: Net-(C54-Pad1) -> /Poe/RX_N
- C44 pad 2: Net-(J2-RD-) -> /Poe/RX_N
- C58 pad 1: /MCU/CELL_STATUS -> /Expander/CELL_STATUS
- J11 pad 10: /Outputs/MM_TX -> /MCU/MM_TX
- J11 pad 11: /Outputs/MM_RTS -> /MCU/MM_RTS
- J11 pad 12: /Outputs/MM_CTS -> /MCU/MM_CTS
- J11 pad 13: /Outputs/~{MM_RST} -> /Expander/~{MM_RST}
- J11 pad 14: /Outputs/SPARE1 -> /Expander/SPARE2
- J11 pad 15: /Outputs/SPARE2 -> /Expander/SPARE1
- J11 pad 6: /Outputs/LED1 -> /MCU/LED1
- J11 pad 7: /Outputs/LED2 -> /MCU/LED2
- J11 pad 8: /Outputs/LED3 -> /MCU/LED3
- J11 pad 9: /Outputs/MM_RX -> /MCU/MM_RX
- J12 pad 2: /Outputs/~{MM_RST} -> /Expander/~{MM_RST}
- J12 pad 3: /Outputs/MM_SOP -> /Expander/MM_SOP
- J12 pad 4: /Outputs/MM_RX -> /MCU/MM_RX
- J12 pad 7: /Outputs/MM_TX -> /MCU/MM_TX
- J12 pad 8: /Outputs/MM_SYNC -> /Expander/MM_SYNC
- J2 pad 3: Net-(J2-RD-) -> /Poe/RX_N
- J2 pad 5: Net-(J2-RD+) -> /Poe/RX_P
- J5 pad 5: /Expander/CAM_SD_SCK -> /Expander/CAM_SD_SCLK
- J7 pad 3: /Outputs/CAM_SD_SCLK -> /Expander/CAM_SD_SCLK
- J7 pad 4: /Outputs/CAM_SD_MISO -> /Expander/CAM_SD_MISO
- J7 pad 5: /Outputs/CAM_SD_MOSI -> /Expander/CAM_SD_MOSI
- J7 pad 6: /Outputs/~{CAM_CS} -> /MCU/~{CAM_CS}
- Q4 pad 1: /MCU/CELL_ON_OFF -> /Expander/CELL_ON_OFF
- Q5 pad 3: /MCU/CELL_STATUS -> /Expander/CELL_STATUS
- R34 pad 1: Net-(U9-RXN) -> /Poe/RX_N
- R34 pad 2: Net-(C54-Pad1) -> /Poe/RX_N
- R35 pad 1: /Poe/RXP -> /Poe/RX_P
- R35 pad 2: /Poe/RXP -> /Poe/RX_P
- R37 pad 2: /Poe/RXP -> /Poe/RX_P
- R39 pad 2: Net-(C54-Pad1) -> /Poe/RX_N
- R4 pad 2: Net-(C4-Pad1) -> Net-(U2-VCC)
- R52 pad 2: /MCU/CELL_RST -> /Expander/CELL_RST
- R56 pad 1: /MCU/WD_DONE -> /Expander/WD_DONE
- R59 pad 2: /MCU/CELL_STATUS -> /Expander/CELL_STATUS
- R66 pad 2: /Outputs/BUZZ -> /MCU/BUZZ/USB-
- R68 pad 2: /Outputs/STROBE -> /MCU/STROBE/USB+
- TP14 pad 1: /MCU/CELL_ON_OFF -> /Expander/CELL_ON_OFF
- U12 pad 20: unconnected-(U5-GPA3-Pad20) -> /Expander/DF_BUSY
- U12 pad 21: unconnected-(U5-GPA4-Pad21) -> /Expander/SPARE1
- U12 pad 22: unconnected-(U5-GPA5-Pad22) -> /Expander/SPARE2
- U12 pad 26: /Expander/~{RSTn} -> /Expander/ETH_RST
- U12 pad 8: /Expander/SCL -> /MCU/SCL
- U12 pad 9: /Expander/SDA -> /MCU/SDA
- U13 pad 16: /Outputs/DF_BUSY -> /Expander/DF_BUSY
- U13 pad 2: /Outputs/DF_RX -> /MCU/DF_RX
- U13 pad 3: /Outputs/DF_TX -> /MCU/DF_TX
- U2 pad 6: unconnected-(U2-VCC-Pad6) -> Net-(U2-VCC)
- U7 pad 32: /Poe/~{SCSn} -> /MCU/~{ETH_CS}
- U7 pad 33: /Poe/SCLK -> /MCU/ETH_SCLK
- U7 pad 34: /Poe/MISO -> /MCU/ETH_MOSI
- U7 pad 35: /Poe/MOSI -> /MCU/ETH_MISO
- U7 pad 36: /Poe/~{INTn} -> /MCU/~{ETH_INT}
- U7 pad 37: /Poe/~{RSTn} -> /Expander/ETH_RST
- U7 pad 5: Net-(U9-RXN) -> /Poe/RX_N
- U7 pad 6: /Poe/RXP -> /Poe/RX_P
- U8 pad 13: /MCU/USB- -> /MCU/BUZZ/USB-
- U8 pad 14: /MCU/USB+ -> /MCU/STROBE/USB+
- U8 pad 18: /MCU/ETH_CS -> /MCU/~{ETH_CS}
- U8 pad 26: /MCU/~{IO_RST} -> /Expander/~{IO_RST}
- U8 pad 31: /MCU/CAM_SD_CLK -> /Expander/CAM_SD_SCLK
- U8 pad 32: /MCU/CAM_SD_MOSI -> /Expander/CAM_SD_MOSI
- U8 pad 33: /MCU/CAM_SD_MISO -> /Expander/CAM_SD_MISO
- U8 pad 35: /MCU/~{SD_CS} -> /Expander/~{SD_CS}
- U8 pad 7: /MCU/~{INTn} -> /MCU/~{ETH_INT}
- U9 pad 4: /MCU/WD_DONE -> /Expander/WD_DONE
Routing:
- net /Poe/RX_P: track 0.00 -> 25.3 mm
- net /Poe/RX_N: track 0.00 -> 25.2 mm
- net /Poe/TX_N: track 0.00 -> 17.8 mm
- net /Poe/TX_P: track 0.00 -> 17.7 mm
- net Net-(J2-RCT): track 0.00 -> 11.2 mm, vias 0 -> 2
- net Net-(J2-TCT): track 0.00 -> 8.39 mm
- net Net-(U7-XO): track 0.00 -> 4.66 mm
- net Net-(U7-PMODE2): track 0.00 -> 4.63 mm
- net Net-(U7-PMODE0): track 0.00 -> 4.55 mm
- net Net-(U7-PMODE1): track 0.00 -> 4.23 mm
- net /Poe/EXRES1: track 0.00 -> 4.22 mm
- net Net-(U7-XI): track 0.00 -> 2.83 mm
- net /Poe/ACTLED: track 0.00 -> 1.90 mm, vias 0 -> 1
- net /Poe/LINKLED: track 0.00 -> 1.45 mm, vias 0 -> 1
Other:
- copper layers 2 -> 4

Commit message: wip - still working on layout
Parts:
- moved C49 57.1 mm to (89.4, 87.5)
- moved D7 57.1 mm to (90.3, 89.5)
- moved R51 57.1 mm to (89.4, 85.9)
- moved S1 57.1 mm to (84.4, 86.3)
- moved IC2 57.0 mm to (162.8, 93.6), turned to 0 degrees
- moved TP8 56.6 mm to (87.5, 92.4)
- moved R48 54.7 mm to (134.1, 108.2)
- moved J4 54.7 mm to (140.0, 107.0)
- moved Q2 54.7 mm to (134.9, 103.7)
- moved R47 54.7 mm to (134.1, 106.6)
- moved D4 48.4 mm to (151.2, 98.5), turned to 180 degrees
- moved C52 19.6 mm to (157.1, 76.0), turned to 90 degrees
- moved C25 19.2 mm to (166.8, 84.0), turned to -90 degrees
- moved C32 18.9 mm to (166.5, 65.6)
- moved C30 18.8 mm to (164.3, 65.6)
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Routing:
- net /Poe/POE+: track 0.00 -> 47.5 mm, vias 0 -> 19
- net Net-(IC3-IN4): track 0.00 -> 30.4 mm
- net GND: track 0.00 -> 26.1 mm, vias 0 -> 14
- net Net-(U2-FB): track 0.00 -> 24.6 mm, vias 0 -> 2
- net Net-(IC3-IN3): track 0.00 -> 24.3 mm
- net Net-(U1-CDB): track 0.00 -> 22.9 mm, vias 0 -> 2
- net Net-(IC3-IN2): track 0.00 -> 20.1 mm
- net +3V9: track 0.00 -> 19.7 mm, vias 0 -> 2
- net /Poe/POE-: track 0.00 -> 16.7 mm, vias 0 -> 13
- net +5VP: track 0.00 -> 15.4 mm
- net Net-(IC3-IN1): track 0.00 -> 14.3 mm
- net Net-(U2-VCC): track 0.00 -> 12.7 mm
- net Net-(U3-FB): track 0.00 -> 11.9 mm
- net Net-(U2-PG): track 0.00 -> 11.4 mm
- net Net-(F1-Pad1): track 0.00 -> 10.5 mm
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- added copper zone on B.Cu, net +12VDC
- added copper zone on In2.Cu, net +12VDC
- added copper zone on B.Cu, net +12VP
- added copper zone on In2.Cu, net +12VP
- added copper zone on B.Cu, net +3V3
- added copper zone on In2.Cu, net +3V3
- added copper zone on B.Cu, net +3V9
- added copper zone on B.Cu, net +5V
- added copper zone on In2.Cu, net +5V
- added copper zone on B.Cu, net +5VDC
- added copper zone on In2.Cu, net +5VDC
- added copper zone on B.Cu, net +5VP
- added copper zone on B.Cu, net /Poe/POE+
- added copper zone on In2.Cu, net /Poe/POE+
- added copper zone on B.Cu, net /Poe/POE-
- added copper zone on In2.Cu, net /Poe/POE-
- added copper zone on B.Cu, net GND
- added copper zone on In1.Cu, net GND
- added copper zone on B.Cu, net Net-(D3-PadA)
- added copper zone on B.Cu, net Net-(D5-K)
- added copper zone on B.Cu, net Net-(D6-K)
- added copper zone on B.Cu, net Net-(U2-SW)
- added copper zone on B.Cu, net Net-(U5-SW)
- added copper zone on B.Cu, net Net-(U6-SW)

Commit message: checkpoint
Parts:
- C49, D7, R51: moved to F.Cu
- moved S1 60.7 mm to (141.6, 106.7), turned to 0 degrees
- moved D7 59.2 mm to (147.2, 105.8), turned to -90 degrees
- moved C49 55.9 mm to (142.4, 105.3), turned to -90 degrees
- moved R51 54.9 mm to (140.7, 105.3), turned to 90 degrees
- moved J4 20.0 mm to (145.6, 87.8), turned to 90 degrees
- moved R48 19.9 mm to (147.0, 93.0), turned to 90 degrees
- moved TP5 19.7 mm to (158.4, 88.4)
- moved TP8 18.4 mm to (86.8, 74.0)
- moved R47 17.7 mm to (145.4, 93.0), turned to 90 degrees
- moved Q2 13.8 mm to (142.5, 92.2), turned to 90 degrees
- moved J10 7.41 mm to (125.7, 95.5)
Routing:
- net +5VP: track 15.4 -> 61.7 mm, vias 0 -> 2
- net Net-(U1-CDB): track 22.9 -> 59.3 mm, vias 2 -> 4
- net Net-(D6-K): track 0.00 -> 18.1 mm
- net +3V3: track 4.22 -> 18.0 mm, vias 16 -> 24
- net Net-(IC3-IN3): track 24.3 -> 11.3 mm
- net GND: track 26.1 -> 38.6 mm, vias 14 -> 20
- net Net-(C13-Pad2): track 0.00 -> 6.23 mm
- net /MCU/~{EN_RST}: track 0.00 -> 3.40 mm
- net Net-(R10-Pad1): track 5.80 -> 8.86 mm
- net Net-(U4-BS): track 0.00 -> 2.37 mm
- net Net-(C9-Pad1): track 0.00 -> 2.22 mm
- net Net-(IC3-IN4): track 30.4 -> 29.3 mm
- net +12VDC: vias 8 -> 12
- added copper zone on B.Cu, net +12V
- added copper zone on F.Cu, net GND
- added copper zone on B.Cu, net Net-(F1-Pad1)
- added copper zone on B.Cu, net Net-(IC3-IN1)
- added copper zone on B.Cu, net Net-(IC3-IN2)
- added copper zone on B.Cu, net Net-(IC3-IN3)
- added copper zone on B.Cu, net Net-(IC3-IN4)
